File: PaletteMux.kicad_sch (KiCad schematic)
At the start: 21 parts, among them U42 74LS138, U43 CD4066BM, U44 CD4066BM, U45 CD4066BM, U46 CD4066BM, U47 CD4066BM, U48 CD4066BM, U49 CD4066BM, U50 CD4066BM, U51 CD4066BM, U52 CD4066BM, U53 CD4066BM, U54 CD4066BM, U55 CD4066BM, U56 CD4066BM, U57 CD4066BM, U58 CD4066BM, U60 4053, U61 74LS21, U62 74LS138, U63 74LS138

Commit message: introduce PDF output from schematics
Connections:
- net +5V: now also U61.14 (VCC)
- net GND: now also U61.7 (GND)
Other:
- moved on the sheet: U42, U43D, U43E, U44D, U44E, U45D, U45E, U46D, U46E, U47D, U47E, U48D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
