File: DIY-Video.kicad_pcb (KiCad board)
At the start: 4 copper layers, 258.4 x 142.5 mm, 162 parts, among them J1 VIDEO IO, J2 Host Address Bus, J3 Host Data Bus, J4 Host Control Bus, U1 74LS163, U10 74LS30, U11 74LS00, U12 74LS30, U13 74LS20, U14 74LS14, U15 74LS30, U16 74LS20, U17 74LS30, U18 74LS00, U19 74LS32, U2 74LS163, U20 74LS30, U21 74LS163, U22 74LS253, U23 74LS163, U24 74LS253, U25 74LS14, U26 74LS163, U27 74LS253, U28 74LS163, U29 74LS253, U3 74LS163, U30 74LS373, U31 74LS163, U32 74LS138, U33 74LS151, U34 74LS151, U35 74LS151, U36 74LS151, U37 74LS151, U38 74LS151, U39 74LS151, U4 74LS163, U40 74LS352, U41 74LS352, U42 74LS138, U43 CD4066BM, U44 CD4066BM, U45 CD4066BM, U46 CD4066BM, U47 CD4066BM, U48 CD4066BM, U49 CD4066BM, U5 74LS163, U50 CD4066BM, U51 CD4066BM, U52 CD4066BM, U53 CD4066BM, U54 CD4066BM, U55 CD4066BM, U56 CD4066BM, U57 CD4066BM, U58 CD4066BM, U59 74LS00, U6 74LS163, U60 4053, U61 74LS21, U62 74LS138, U63 74LS138, U64 74LS30, U65 74LS20, U66 74LS00, U67 74LS32, U68 74LS148, U69 74LS30, U7 74LS20, U70 74LS245, U71 CY62256-70PC, U72 74LS244, U73 74LS244, U74 74LS244, U75 74LS244, U76 74LS04, U77 74LS244, U78 74LS163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

Commit message: isolate each schematic function for testing
Parts:
- added IC26: MC6821, Package_DIP:DIP-40_W15.24mm, F.Cu at (-110.0, 23.6)
- added J10: PosResets, Connector_PinSocket_2.54mm:PinSocket_1x04_P2.54mm_Vertical, B.Cu at (63.3, 156.5)
- added J11: Power and Clock, Connector_PinSocket_2.54mm:PinSocket_1x04_P2.54mm_Vertical, B.Cu at (30.1, 104.5)
- added J5: posX, Connector_PinSocket_2.54mm:PinSocket_1x10_P2.54mm_Vertical, B.Cu at (78.4, 105.7)
- added J6: posY, Connector_PinSocket_2.54mm:PinSocket_1x10_P2.54mm_Vertical, B.Cu at (78.4, 133.6)
- added J7: ViewportTriggers, Connector_PinSocket_2.54mm:PinSocket_1x06_P2.54mm_Vertical, B.Cu at (121.5, 117.1)
- added J8: posX, Connector_PinSocket_2.54mm:PinSocket_1x10_P2.54mm_Vertical, B.Cu at (68.1, 105.7)
- added J9: posY, Connector_PinSocket_2.54mm:PinSocket_1x10_P2.54mm_Vertical, B.Cu at (68.1, 133.6)
- added U100: 74LS374, Package_SO:SO-20_5.3x12.6mm_P1.27mm, F.Cu at (-69.1, 28.7)
- added U101: 74LS374, Package_SO:SO-20_5.3x12.6mm_P1.27mm, F.Cu at (-58.6, 28.7)
- added U102: 74LS163, Package_SO:SOIC-16_3.9x9.9mm_P1.27mm, F.Cu at (-70.1, 41.7)
- added U110: 74LS08, Package_SO:SO-14_3.9x8.65mm_P1.27mm, F.Cu at (38.1, 141.6)
- added U111: 74LS30, Package_SO:SO-14_3.9x8.65mm_P1.27mm, F.Cu at (38.1, 117.4)
- added U112: 74LS30, Package_SO:SO-14_3.9x8.65mm_P1.27mm, F.Cu at (86.5, 109.5)
- added U113: 74LS30, Package_SO:SO-14_3.9x8.65mm_P1.27mm, F.Cu at (96.3, 131.1)
- added U114: 74LS00, Package_SO:SO-14_3.9x8.65mm_P1.27mm, F.Cu at (105.9, 120.3)
- added U115: 74LS32, Package_SO:SO-14_3.9x8.65mm_P1.27mm, F.Cu at (115.3, 120.3)
- added U118: 74LS04, Package_SO:SOIC-14_3.9x8.7mm_P1.27mm, F.Cu at (84.7, 95.1)
- added U119: 74LS08, Package_SO:SOIC-14_3.9x8.7mm_P1.27mm, F.Cu at (115.3, 142.0)
- added U121: 74LS163, Package_SO:SOIC-16_3.9x9.9mm_P1.27mm, F.Cu at (-89.0, 27.4)
- added U122: 74LS163, Package_SO:SOIC-16_3.9x9.9mm_P1.27mm, F.Cu at (-80.5, 27.4)
- U14, U8: value 74LS14 -> 74LS04
- U40, U41: value 74LS352 -> 74LS153
- U7: value 74LS20 -> 74LS30
- moved J4 361.0 mm to (-84.7, 47.0)
- moved U90 119.3 mm to (-59.0, 43.2)
- moved R11 67.3 mm to (118.7, 94.1)
- moved U59 67.3 mm to (112.8, 84.0)
- moved U64 67.3 mm to (121.3, 84.0)
- moved U65 67.3 mm to (129.7, 84.0)
- moved U67 67.3 mm to (129.8, 94.6)
- moved U69 67.3 mm to (138.4, 84.0)
- moved R10 67.3 mm to (118.7, 92.1)
- moved R9 67.3 mm to (118.7, 90.1)
- moved U68 67.3 mm to (112.8, 95.2)
- moved U83 67.3 mm to (138.4, 94.6)
- moved U14 49.7 mm to (86.5, 131.1)
- moved U60 48.1 mm to (269.4, 32.1), turned to 0 degrees
- moved U12 44.5 mm to (96.3, 109.4)
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Connections:
- net /ControlRegisters/RR0 renamed /BitmapAddressRegister/RR0
- net /ControlRegisters/RR1 renamed /BitmapAddressRegister/RR1
- net Net-(U88-O5) renamed /ControlRegisters/External
- net Net-(U88-O6) renamed /ControlRegisters/ExtTriggerHi/~{Lo}
- net Net-(U88-O7) renamed /ControlRegisters/EnExternalTrigger
- net Net-(U96-O0) renamed /ControlRegisters/EnableTile
- net Net-(U96-O1) renamed /ControlRegisters/EnableSprite
- net Net-(U96-O2) renamed /ControlRegisters/FontMap0
- net Net-(U96-O3) renamed /ControlRegisters/FontMap1
- U11 pad 1: /ViewPort/HEnd -> /ViewPort/NTSCVStart
- U11 pad 2: Net-(U11-Pad2) -> /ViewPort/~{NTSCVCountEnable}
- U11 pad 5: /ViewPort/HStart -> /ViewPort/NTSCVEnd
- U11 pad 6: Net-(U11-Pad2) -> /ViewPort/~{NTSCVCountEnable}
- U13 pad 10: /FrameTiming/Y6 -> /FrameTiming/X5
- U13 pad 12: /ViewPort/~{Y7} -> /FrameTiming/X6
- U13 pad 13: /ViewPort/~{Y8} -> /FrameTiming/X8
- U13 pad 8: /ViewPort/PALVStart -> Net-(U114-Pad1)
- U13 pad 9: /FrameTiming/Y3 -> /FrameTiming/X2
- U16 pad 10: /FrameTiming/X5 -> /FrameTiming/Y6
- U16 pad 12: /FrameTiming/X6 -> /ViewPort/~{Y7}
- U16 pad 13: /FrameTiming/X8 -> /ViewPort/~{Y8}
- U16 pad 8: Net-(U16-Pad8) -> /ViewPort/PALVStart
- U16 pad 9: /FrameTiming/X2 -> /FrameTiming/Y3
- U18 pad 1: /ViewPort/NTSCVStart -> /ViewPort/HEnd
- U18 pad 12: Net-(U18-Pad12) -> Net-(U115-Pad1)
- U18 pad 3: /ViewPort/~{NTSCVCountEnable} -> Net-(U115-Pad4)
- U18 pad 4: /ViewPort/~{NTSCVCountEnable} -> Net-(U115-Pad4)
- U18 pad 5: /ViewPort/NTSCVEnd -> /ViewPort/HStart
- U18 pad 8: Net-(U18-Pad12) -> Net-(U115-Pad1)
- U18 pad 9: Net-(U16-Pad8) -> Net-(U112-Pad8)
- U19 pad 1: /ViewPort/~{NTSCVCountEnable} -> Format
- U19 pad 11: ~{HLoadEnable} -> unconnected-(U19-Pad11)
- U19 pad 12: Net-(U18-Pad12) -> unconnected-(U19-Pad12)
- U19 pad 13: ~{VCountEnable} -> unconnected-(U19-Pad13)
- U19 pad 2: Format -> /ViewPort/~{NTSCVCountEnable}
- U19 pad 3: Net-(U19-Pad3) -> Net-(U119-Pad5)
- U19 pad 4: Net-(U19-Pad4) -> unconnected-(U19-Pad4)
- U19 pad 5: Net-(U19-Pad3) -> unconnected-(U19-Pad5)
- U19 pad 6: ~{VCountEnable} -> unconnected-(U19-Pad6)
- U19 pad 8: Net-(U19-Pad4) -> Net-(U119-Pad4)
- U2 pad 10: /PositionCounters/CX0 -> +5V
- U2 pad 2: 14M -> /PositionCounters/CX0
- U20 pad 1: /FrameTiming/X2 -> /FrameTiming/X1
- U20 pad 2: /FrameTiming/X5 -> /FrameTiming/X2
- U20 pad 3: /ViewPort/~{X7} -> /FrameTiming/X5
- U20 pad 4: /ViewPort/~{X8} -> /ViewPort/~{X7}
- U20 pad 5: /ViewPort/~{X9} -> /ViewPort/~{X8}
- U20 pad 6: +5V -> /ViewPort/~{X9}
- U22 pad 1: /BitmapDataCounter/LoadEnable -> ~{HLoadEnable}
- U22 pad 15: GND -> +5V
- U24 pad 1: +5V -> GND
- U24 pad 15: GND -> +5V
- U27 pad 1: /BitmapPixelCounter/CountEnable -> ~{HCountEnable}
- U27 pad 15: GND -> +5V
- U29 pad 1: +5V -> GND
- U29 pad 15: GND -> +5V
- U3 pad 10: /PositionCounters/CX1 -> +5V
- U3 pad 2: 14M -> /PositionCounters/CX1
- U31 pad 1: GND -> +5V
- U31 pad 3: GND -> +5V
- U31 pad 4: GND -> +5V
- U31 pad 5: GND -> +5V
- U31 pad 6: GND -> +5V
- U31 pad 9: GND -> /BitmapPixelData/~{MR}
- U33 pad 1: /BitmapPixelData/D3 -> /BitmapPixelData/D4
- U33 pad 12: /BitmapPixelData/D7 -> /BitmapPixelData/D0
- U33 pad 13: /BitmapPixelData/D6 -> /BitmapPixelData/D1
- U33 pad 14: /BitmapPixelData/D5 -> /BitmapPixelData/D2
- U33 pad 15: /BitmapPixelData/D4 -> /BitmapPixelData/D3
- U33 pad 2: /BitmapPixelData/D2 -> /BitmapPixelData/D5
- U33 pad 3: /BitmapPixelData/D1 -> /BitmapPixelData/D6
- U33 pad 4: /BitmapPixelData/D0 -> /BitmapPixelData/D7
- U34 pad 1: /BitmapPixelData/D6 -> /BitmapPixelData/D0
- U34 pad 2: /BitmapPixelData/D4 -> /BitmapPixelData/D2
- U34 pad 3: /BitmapPixelData/D2 -> /BitmapPixelData/D4
- U34 pad 4: /BitmapPixelData/D0 -> /BitmapPixelData/D6
- U35 pad 1: /BitmapPixelData/D7 -> /BitmapPixelData/D1
- U35 pad 2: /BitmapPixelData/D5 -> /BitmapPixelData/D3
- U35 pad 3: /BitmapPixelData/D3 -> /BitmapPixelData/D5
- U35 pad 4: /BitmapPixelData/D1 -> /BitmapPixelData/D7
- U36 pad 3: /BitmapPixelData/D4 -> /BitmapPixelData/D0
- U36 pad 4: /BitmapPixelData/D0 -> /BitmapPixelData/D4
- U37 pad 3: /BitmapPixelData/D5 -> /BitmapPixelData/D1
- U37 pad 4: /BitmapPixelData/D1 -> /BitmapPixelData/D5
- U38 pad 3: /BitmapPixelData/D6 -> /BitmapPixelData/D2
- U38 pad 4: /BitmapPixelData/D2 -> /BitmapPixelData/D6
- U39 pad 3: /BitmapPixelData/D7 -> /BitmapPixelData/D3
- U39 pad 4: /BitmapPixelData/D3 -> /BitmapPixelData/D7
- U4 pad 2: ~{ResetX} -> /PositionCounters/ResetX
- U41 pad 6: GND -> /BitmapPixelData/DefaultPalette1
- U5 pad 10: /PositionCounters/CY0 -> +5V
- U5 pad 2: ~{ResetX} -> /PositionCounters/CY0
- U6 pad 10: /PositionCounters/CY1 -> +5V
- U6 pad 2: ~{ResetX} -> /PositionCounters/CY1
- U61 pad 14: unconnected-(U61C-VCC-Pad14) -> +5V
- U61 pad 7: unconnected-(U61C-GND-Pad7) -> GND
- U69 pad 14: (no net) -> +5V
- U69 pad 7: (no net) -> GND
- U7 pad 10: /FrameTiming/Y1 -> (no net)
- U7 pad 11: (no net) -> /FrameTiming/Y8
- U7 pad 12: /FrameTiming/Y6 -> /FrameTiming/Y2
- U7 pad 13: /FrameTiming/Y8 -> (no net)
- U7 pad 2: /FrameTiming/Y1 -> +5V
- U7 pad 3: (no net) -> /FrameTiming/Y0
- U7 pad 4: /FrameTiming/Y2 -> +5V
- U7 pad 5: /FrameTiming/Y8 -> +5V
- U7 pad 6: /PositionCounters/NTSC_RY -> +5V
- U7 pad 8: /PositionCounters/PAL_RY -> /PositionCounters/NTSC_RY
- U7 pad 9: +5V -> (no net)
- U76 pad 13: unconnected-(U76-Pad13) -> +5V
- U76 pad 14: unconnected-(U76G-VCC-Pad14) -> +5V
- U76 pad 7: unconnected-(U76G-GND-Pad7) -> GND
- U78 pad 3: GND -> /BitmapAddressRegister/RA0
- U78 pad 4: GND -> /BitmapAddressRegister/RA1
- U78 pad 5: GND -> /BitmapAddressRegister/RA2
- U78 pad 6: GND -> /BitmapAddressRegister/RA3
- U78 pad 9: GND -> /BitmapAddressRegister/Reload
- U79 pad 3: GND -> /BitmapAddressRegister/RA4
- U79 pad 4: GND -> /BitmapAddressRegister/RA5
- U79 pad 5: GND -> /BitmapAddressRegister/RA6
- U79 pad 6: GND -> /BitmapAddressRegister/RA7
- U79 pad 9: GND -> /BitmapAddressRegister/Reload
- U8 pad 12: /BitmapDataCounter/LoadEnable -> unconnected-(U8-Pad12)
- U8 pad 13: ~{HLoadEnable} -> unconnected-(U8-Pad13)
- U8 pad 8: unconnected-(U8-Pad8) -> /PositionCounters/ResetX
- U8 pad 9: unconnected-(U8-Pad9) -> ~{ResetX}
- U80 pad 3: GND -> /BitmapAddressRegister/RA8
- U80 pad 4: GND -> /BitmapAddressRegister/RA9
- U80 pad 5: GND -> /BitmapAddressRegister/RA10
- U80 pad 6: GND -> /BitmapAddressRegister/RA11
- U80 pad 9: GND -> /BitmapAddressRegister/Reload
- U81 pad 3: GND -> /BitmapAddressRegister/RA12
- U81 pad 4: GND -> /BitmapAddressRegister/RA13
- U81 pad 5: GND -> /BitmapAddressRegister/RA14
- U81 pad 9: GND -> /BitmapAddressRegister/Reload
- U84 pad 12: /ControlRegisters/BPP0 -> /BitmapDataCounter/BPP0
- U84 pad 15: /ControlRegisters/BPP1 -> /BitmapDataCounter/BPP1
- U84 pad 16: /ControlRegisters/CPP0 -> /BitmapDataCounter/CPP0
- U84 pad 19: /ControlRegisters/CPP1 -> /BitmapDataCounter/CPP1
- U85 pad 11: /ControlRegisters/BPP0 -> /BitmapDataCounter/BPP0
- U85 pad 13: /ControlRegisters/BPP1 -> /BitmapDataCounter/BPP1
- U85 pad 15: /ControlRegisters/CPP0 -> /BitmapDataCounter/CPP0
- U85 pad 17: /ControlRegisters/CPP1 -> /BitmapDataCounter/CPP1
- U9 pad 10: Net-(U9-Pad10) -> unconnected-(U9-Pad10)
- U9 pad 11: ~{HCountEnable} -> unconnected-(U9-Pad11)
- U9 pad 12: Net-(U11-Pad3) -> unconnected-(U9-Pad12)
- U9 pad 13: ~{VCountEnable} -> unconnected-(U9-Pad13)
- U9 pad 3: Net-(U9-Pad3) -> Net-(U110-Pad12)
- U9 pad 6: Net-(U9-Pad10) -> Net-(U110-Pad13)
- U9 pad 8: ~{ResetY} -> unconnected-(U9-Pad8)
- U9 pad 9: Net-(U9-Pad3) -> unconnected-(U9-Pad9)
- U90 pad 1: (no net) -> unconnected-(U90-Pad1)
- U90 pad 2: (no net) -> unconnected-(U90-Pad2)
- U90 pad 3: (no net) -> unconnected-(U90-Pad3)
- U93 pad 14: unconnected-(U93E-VCC-Pad14) -> +5V
- U93 pad 7: unconnected-(U93E-GND-Pad7) -> GND
- U94 pad 14: unconnected-(U94E-VCC-Pad14) -> +5V
- U94 pad 7: unconnected-(U94E-GND-Pad7) -> GND
- U95 pad 14: unconnected-(U95E-VCC-Pad14) -> +5V
- U95 pad 7: unconnected-(U95E-GND-Pad7) -> GND
- U98 pad 10: unconnected-(U98-Pad10) -> GND
- U98 pad 12: unconnected-(U98-Pad12) -> GND
- U98 pad 13: unconnected-(U98-Pad13) -> GND
- U98 pad 14: unconnected-(U98E-VCC-Pad14) -> +5V
- U98 pad 7: unconnected-(U98E-GND-Pad7) -> GND
- U98 pad 9: unconnected-(U98-Pad9) -> GND
- U99 pad 14: unconnected-(U99E-VCC-Pad14) -> +5V
- U99 pad 7: unconnected-(U99E-GND-Pad7) -> GND
Routing:
- net /FrameTiming/Y5: track 0.00 -> 121.8 mm, vias 0 -> 4
- net /FrameTiming/X5: track 20.1 -> 122.6 mm, vias 0 -> 5
- net /FrameTiming/Y4: track 0.00 -> 99.8 mm, vias 0 -> 2
- net /FrameTiming/Y8: track 37.6 -> 131.5 mm, vias 0 -> 6
- net /FrameTiming/Y7: track 0.00 -> 91.9 mm, vias 0 -> 5
- net /FrameTiming/X2: track 45.9 -> 132.1 mm, vias 0 -> 5
- net /FrameTiming/X6: track 21.1 -> 104.7 mm, vias 0 -> 4
- net /FrameTiming/Y0: track 11.0 -> 94.4 mm, vias 0 -> 4
- net /FrameTiming/Y1: track 22.9 -> 105.3 mm, vias 0 -> 6
- net /FrameTiming/Y2: track 14.2 -> 90.4 mm, vias 0 -> 3
- net /FrameTiming/X1: track 0.00 -> 71.8 mm, vias 0 -> 2
- net /FrameTiming/X3: track 17.1 -> 88.8 mm, vias 0 -> 2
- net /FrameTiming/X8: track 63.1 -> 127.4 mm, vias 2 -> 5
- net /FrameTiming/X4: track 11.8 -> 75.7 mm, vias 0 -> 2
- net /FrameTiming/Y6: track 24.6 -> 83.8 mm, vias 0 -> 5
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Other:
- board text added: "Analog Output"
- board text added: "Viewport"
- board text added: "X-Y Counters"

Commit message: rework schematic isolation
Parts:
- removed U91, U92: 74LS21, Package_SO:SO-14_3.9x8.65mm_P1.27mm
- removed U95, U99: 74LS32, Package_SO:SO-14_3.9x8.65mm_P1.27mm
- added J12: posX, Connector_PinSocket_2.54mm:PinSocket_1x10_P2.54mm_Vertical, B.Cu at (136.9, 105.6)
- added J13: posY, Connector_PinSocket_2.54mm:PinSocket_1x10_P2.54mm_Vertical, B.Cu at (136.9, 133.6)
- added J14: TimingTriggers, Connector_PinSocket_2.54mm:PinSocket_1x06_P2.54mm_Vertical, B.Cu at (142.0, 156.4)
- added J15: ViewportOutput, Connector_PinSocket_2.54mm:PinSocket_1x06_P2.54mm_Vertical, B.Cu at (180.6, 142.9)
- added J16: Power and Clock, Connector_PinSocket_2.54mm:PinSocket_1x04_P2.54mm_Vertical, B.Cu at (199.6, 104.9)
- added J17: Triggers, Connector_PinSocket_2.54mm:PinSocket_1x04_P2.54mm_Vertical, B.Cu at (243.2, 108.0)
- added J18: OpMode, Connector_PinSocket_2.54mm:PinSocket_1x04_P2.54mm_Vertical, B.Cu at (230.4, 104.9)
- added J19: XDBus, Connector_PinHeader_1.27mm:PinHeader_1x08_P1.27mm_Vertical, B.Cu at (99.2, -5.84)
- added J20: XDBus, Connector_PinHeader_1.27mm:PinHeader_1x08_P1.27mm_Vertical, B.Cu at (128.7, -5.84)
- added J21: Register0, Connector_PinHeader_1.27mm:PinHeader_1x10_P1.27mm_Vertical, B.Cu at (113.9, -6.35)
- added J22: XDBus, Connector_PinHeader_1.27mm:PinHeader_1x08_P1.27mm_Vertical, B.Cu at (99.2, 11.9)
- added J23: XDBus, Connector_PinHeader_1.27mm:PinHeader_1x08_P1.27mm_Vertical, B.Cu at (128.7, 11.9)
- added J24: Register2, Connector_PinHeader_1.27mm:PinHeader_1x10_P1.27mm_Vertical, B.Cu at (113.9, 11.4)
- added J25: XDBus, Connector_PinHeader_1.27mm:PinHeader_1x08_P1.27mm_Vertical, B.Cu at (99.2, 29.2)
- added J26: XDBus, Connector_PinHeader_1.27mm:PinHeader_1x08_P1.27mm_Vertical, B.Cu at (128.4, 29.2)
- added J27: Register1, Connector_PinHeader_1.27mm:PinHeader_1x10_P1.27mm_Vertical, B.Cu at (113.9, 28.7)
- added J28: XDBus, Connector_PinHeader_1.27mm:PinHeader_1x08_P1.27mm_Vertical, B.Cu at (99.2, 47.8)
- added J29: XDBus, Connector_PinHeader_1.27mm:PinHeader_1x08_P1.27mm_Vertical, B.Cu at (128.4, 47.8)
- added J30: Register3, Connector_PinHeader_1.27mm:PinHeader_1x10_P1.27mm_Vertical, B.Cu at (113.9, 47.2)
- added U127: 74LS04, Package_SO:SOIC-14_3.9x8.7mm_P1.27mm, F.Cu at (171.1, 135.2)
- added U128: 74LS04, Package_SO:SOIC-14_3.9x8.7mm_P1.27mm, F.Cu at (205.8, 130.0)
- added U129: 74LS30, Package_SO:SO-14_3.9x8.65mm_P1.27mm, F.Cu at (146.4, 113.5)
- R10, R11, R9: moved to B.Cu
- U25: value 74LS14 -> 74LS32; footprint Package_SO:SO-14_3.9x8.65mm_P1.27mm -> Package_SO:SOIC-14_3.9x8.7mm_P1.27mm
- U67: value 74LS32 -> 74LS138; footprint Package_SO:SO-14_3.9x8.65mm_P1.27mm -> Package_SO:SOIC-16_3.9x9.9mm_P1.27mm
- moved U42 439.4 mm to (-12.4, 41.7)
- moved U61 439.4 mm to (-65.7, 69.2)
- moved U78 439.4 mm to (-65.7, 82.2)
- moved U79 439.4 mm to (-57.3, 82.2)
- moved U80 439.4 mm to (-48.8, 82.2)
- moved U81 439.4 mm to (-40.4, 82.2)
- moved U30 336.9 mm to (180.7, 63.6)
- moved U31 336.9 mm to (144.6, 62.2)
- moved U32 336.9 mm to (153.1, 62.2)
- moved U33 336.9 mm to (161.5, 62.2)
- moved U35 336.9 mm to (144.6, 73.8)
- moved U36 336.9 mm to (153.1, 73.8)
- moved U37 336.9 mm to (161.5, 73.8)
- moved U39 336.9 mm to (144.6, 85.4)
- moved U40 336.9 mm to (153.1, 85.4)
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Connections:
- net Net-(U96-O4) renamed /ControlRegisters/R3B4
- net Net-(U96-O5) renamed /ControlRegisters/R3B5
- net Net-(U96-O6) renamed /ControlRegisters/R3B6
- net Net-(U96-O7) renamed /ControlRegisters/R3B7
- R10 pad 1: +5V -> ~{Sprite}
- R10 pad 2: ~{Sprite} -> GND
- R11 pad 1: +5V -> ~{Tile}
- R11 pad 2: ~{Tile} -> GND
- R9 pad 1: +5V -> ~{External}
- R9 pad 2: ~{External} -> GND
- U118 pad 14: unconnected-(U118G-VCC-Pad14) -> +5V
- U118 pad 7: unconnected-(U118G-GND-Pad7) -> GND
- U25 pad 1: (no net) -> Net-(U25-Pad1)
- U25 pad 10: ~{Border} -> unconnected-(U25-Pad10)
- U25 pad 11: Net-(U25-Pad11) -> unconnected-(U25-Pad11)
- U25 pad 12: (no net) -> unconnected-(U25-Pad12)
- U25 pad 13: (no net) -> unconnected-(U25-Pad13)
- U25 pad 14: (no net) -> +5V
- U25 pad 2: (no net) -> Net-(U25-Pad2)
- U25 pad 3: (no net) -> Page13
- U25 pad 4: (no net) -> Net-(U25-Pad4)
- U25 pad 5: (no net) -> Net-(U25-Pad5)
- U25 pad 6: (no net) -> Page14
- U25 pad 7: (no net) -> GND
- U25 pad 8: /BitmapPixelCounter/CountEnable -> unconnected-(U25-Pad8)
- U25 pad 9: ~{HCountEnable} -> unconnected-(U25-Pad9)
- U59 pad 1: /FrameTiming/Y5 -> Net-(U59-Pad1)
- U59 pad 12: ~{HSync} -> ~{VSync}
- U59 pad 13: Net-(U59-Pad13) -> ~{ResetY}
- U59 pad 3: ~{VSync} -> ~{HSync}
- U59 pad 4: ~{VSync} -> ~{HSync}
- U59 pad 5: ~{ResetY} -> Net-(U129-Pad8)
- U59 pad 8: ~{HSync} -> ~{VSync}
- U59 pad 9: Net-(U59-Pad9) -> Net-(U127-Pad4)
- U64 pad 11: /FrameTiming/X8 -> /FrameTiming/X9
- U64 pad 12: /FrameTiming/X9 -> /FrameTiming/X8
- U64 pad 3: /FrameTiming/X2 -> +5V
- U64 pad 8: Net-(U59-Pad9) -> Net-(U59-Pad1)
- U65 pad 1: /FrameTiming/X4 -> +5V
- U65 pad 2: /FrameTiming/X5 -> +5V
- U65 pad 4: /FrameTiming/X8 -> ~{VSync}
- U65 pad 5: /FrameTiming/X9 -> ~{HBlank}
- U65 pad 6: Net-(U59-Pad13) -> Net-(U127-Pad11)
- U67 pad 1: ~{VSync} -> /A0
- U67 pad 10: Net-(U67-Pad10) -> /ControlRegisters/~{SelectRegister5}
- U67 pad 11: Page14 -> /ControlRegisters/~{SelectRegister4}
- U67 pad 12: Net-(U67-Pad12) -> /ControlRegisters/~{SelectRegister3}
- U67 pad 13: Net-(U67-Pad13) -> /ControlRegisters/~{SelectRegister2}
- U67 pad 14: +5V -> /ControlRegisters/~{SelectRegister1}
- U67 pad 2: ~{HBlank} -> /A1
- U67 pad 3: ~{Blank} -> /A2
- U67 pad 4: unconnected-(U67-Pad4) -> GND
- U67 pad 5: unconnected-(U67-Pad5) -> GND
- U67 pad 6: unconnected-(U67-Pad6) -> DevSel4
- U67 pad 7: GND -> /ControlRegisters/~{SelectRegister7}
- U67 pad 8: Page13 -> GND
- U67 pad 9: Net-(U67-Pad9) -> /ControlRegisters/~{SelectRegister6}
- U68 pad 1: ~{Border} -> ~{External}
- U68 pad 10: ~{External} -> ~{Border}
- U68 pad 11: ~{Sprite} -> ~{Tile}
- U68 pad 13: ~{Tile} -> ~{Sprite}
- U68 pad 3: ~{VSync} -> ~{HSync}
- U68 pad 4: ~{HSync} -> ~{VSync}
- U69 pad 3: ~{Sprite} -> ~{Blank}
- U69 pad 4: ~{HCountEnable} -> ~{Sprite}
- U69 pad 5: ~{Tile} -> ~{HCountEnable}
- U69 pad 6: ~{Blank} -> ~{Tile}
- U69 pad 8: Net-(U25-Pad11) -> Net-(U127-Pad5)
- U83 pad 3: Net-(U67-Pad9) -> Net-(U25-Pad1)
- U90 pad 11: Net-(U67-Pad13) -> Net-(U25-Pad5)
- U90 pad 6: Net-(U67-Pad10) -> Net-(U25-Pad2)
- U90 pad 8: Net-(U67-Pad12) -> Net-(U25-Pad4)
- U93 pad 1: DevSel4 -> /ControlRegisters/~{SelectRegister1}
- U93 pad 11: Net-(U93-Pad11) -> /ControlRegisters/~{RegisterRead1}
- U93 pad 12: DevSel4 -> /ControlRegisters/~{SelectRegister1}
- U93 pad 13: /ControlRegisters/~{SelectRegister0} -> ~{ExtRead}
- U93 pad 2: /ControlRegisters/~{SelectRegister1} -> ~{ExtWrite}
- U93 pad 3: Net-(U93-Pad3) -> /ControlRegisters/~{RegisterWrite1}
- U93 pad 4: Net-(U93-Pad3) -> /ControlRegisters/~{SelectRegister0}
- U93 pad 9: Net-(U93-Pad11) -> /ControlRegisters/~{SelectRegister0}
- U94 pad 1: Net-(U94-Pad1) -> /ControlRegisters/~{SelectRegister3}
- U94 pad 10: ~{ExtRead} -> ~{ExtWrite}
- U94 pad 11: Net-(U94-Pad11) -> /ControlRegisters/~{RegisterRead3}
- U94 pad 12: DevSel4 -> /ControlRegisters/~{SelectRegister3}
- U94 pad 13: /ControlRegisters/~{SelectRegister1} -> ~{ExtRead}
- U94 pad 3: /ControlRegisters/~{RegisterWrite1} -> /ControlRegisters/~{RegisterWrite3}
- U94 pad 4: DevSel4 -> /ControlRegisters/~{SelectRegister2}
- U94 pad 5: /ControlRegisters/~{SelectRegister0} -> ~{ExtRead}
- U94 pad 6: Net-(U94-Pad1) -> /ControlRegisters/~{RegisterRead2}
- U94 pad 8: /ControlRegisters/~{RegisterRead1} -> /ControlRegisters/~{RegisterWrite2}
- U94 pad 9: Net-(U94-Pad11) -> /ControlRegisters/~{SelectRegister2}
Routing:
- net /XD7: track 4.59 -> 155.7 mm, vias 0 -> 8
- net /XD6: track 4.59 -> 135.3 mm, vias 0 -> 8
- net /XD4: track 4.59 -> 108.0 mm, vias 0 -> 4
- net /XD5: track 4.59 -> 105.3 mm, vias 0 -> 8
- net /FrameTiming/X6: track 104.7 -> 181.4 mm, vias 4 -> 7
- net GND: track 156.4 -> 222.6 mm, vias 113 -> 154
- net ~{VSync}: track 0.00 -> 66.1 mm, vias 0 -> 3
- net Net-(U127-Pad8): track 0.00 -> 65.3 mm, vias 0 -> 2
- net /FrameTiming/X3: track 88.8 -> 153.3 mm
- net ~{ResetX}: track 104.2 -> 164.9 mm
- net /BitmapDataCounter/LoadEnable: track 0.00 -> 57.1 mm
- net /XD3: track 39.9 -> 95.5 mm
- net ~{HSync}: track 0.00 -> 54.4 mm, vias 0 -> 2
- net ~{HLoadEnable}: track 9.42 -> 63.7 mm
- net /XD2: track 39.0 -> 89.8 mm
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Other:
- board size 258.4 x 142.5 mm -> 258.4 x 172.5 mm
- board text added: "Frame Timing"
- board text added: "Pixel Divider"

Commit message: spin register out as separate board
Parts:
- added J31: XDBus, Connector_PinHeader_1.27mm:PinHeader_1x08_P1.27mm_Vertical, B.Cu at (99.0, 58.9)
- added J32: XDBus, Connector_PinHeader_1.27mm:PinHeader_1x08_P1.27mm_Vertical, B.Cu at (128.2, 58.9)
- added J33: Register4, Connector_PinHeader_1.27mm:PinHeader_1x10_P1.27mm_Vertical, B.Cu at (113.7, 58.4)
- added J34: XDBus, Connector_PinHeader_1.27mm:PinHeader_1x08_P1.27mm_Vertical, B.Cu at (99.0, 75.4)
- added J35: XDBus, Connector_PinHeader_1.27mm:PinHeader_1x08_P1.27mm_Vertical, B.Cu at (128.2, 75.4)
- added J36: Register6, Connector_PinHeader_1.27mm:PinHeader_1x10_P1.27mm_Vertical, B.Cu at (113.7, 74.9)
- added J37: XDBus, Connector_PinHeader_1.27mm:PinHeader_1x08_P1.27mm_Vertical, B.Cu at (60.0, 58.9)
- added J38: XDBus, Connector_PinHeader_1.27mm:PinHeader_1x08_P1.27mm_Vertical, B.Cu at (89.2, 58.9)
- added J39: Register5, Connector_PinHeader_1.27mm:PinHeader_1x10_P1.27mm_Vertical, B.Cu at (74.7, 58.4)
- added J40: XDBus, Connector_PinHeader_1.27mm:PinHeader_1x08_P1.27mm_Vertical, B.Cu at (60.0, 75.4)
- added J41: XDBus, Connector_PinHeader_1.27mm:PinHeader_1x08_P1.27mm_Vertical, B.Cu at (89.2, 75.4)
- added J42: Register7, Connector_PinHeader_1.27mm:PinHeader_1x10_P1.27mm_Vertical, B.Cu at (74.7, 74.9)
- added NT49: NetTie_2, NetTie:NetTie-2_SMD_Pad0.5mm, F.Cu at (-96.6, 78.4)
- added U103: 74LS04, Package_SO:SOIC-14_3.9x8.7mm_P1.27mm, F.Cu at (-88.2, 10.5)
- added U104: 74LS21, Package_SO:SOIC-14_3.9x8.7mm_P1.27mm, F.Cu at (-117.5, 10.5)
- added U105: 74LS138, Package_SO:SOIC-16_3.9x9.9mm_P1.27mm, F.Cu at (-117.5, 21.5)
- added U106: 74LS32, Package_SO:SOIC-14_3.9x8.7mm_P1.27mm, F.Cu at (-109.1, 10.5)
- added U107: 74LS138, Package_SO:SOIC-16_3.9x9.9mm_P1.27mm, F.Cu at (-92.2, -2.52)
- added U108: 74LS04, Package_SO:SO-14_3.9x8.65mm_P1.27mm, F.Cu at (-117.5, -3.16)
- added U109: 74LS11, Package_SO:SO-14_3.9x8.65mm_P1.27mm, F.Cu at (-109.1, -3.16)
- added U116: 74LS279, Package_SO:SOIC-16_3.9x9.9mm_P1.27mm, F.Cu at (-83.7, -2.52)
- added U117: 74LS08, Package_SO:SO-14_3.9x8.65mm_P1.27mm, F.Cu at (-77.7, 10.5)
- added U120: 74LS32, Package_SO:SO-14_3.9x8.65mm_P1.27mm, F.Cu at (-100.6, -3.16)
- added U123: 74LS373, Package_SO:SOIC-20W_7.5x12.8mm_P1.27mm, F.Cu at (-115.3, -15.6)
- added U124: 74LS373, Package_SO:SOIC-20W_7.5x12.8mm_P1.27mm, F.Cu at (-102.4, -15.6)
- added U125: 74LS244, Package_SO:SOIC-20W_7.5x12.8mm_P1.27mm, F.Cu at (-89.5, -15.6)
- added U126: 74LS244, Package_SO:SOIC-20W_7.5x12.8mm_P1.27mm, F.Cu at (-76.6, -15.6)
- added U130: 74LS244, Package_SO:SO-20_5.3x12.6mm_P1.27mm, F.Cu at (121.1, 79.4)
- added U131: 74LS374, Package_SO:SO-20_5.3x12.6mm_P1.27mm, F.Cu at (67.4, 62.9)
- added U132: 74LS244, Package_SO:SO-20_5.3x12.6mm_P1.27mm, F.Cu at (81.9, 62.9)
- added U133: 74LS374, Package_SO:SO-20_5.3x12.6mm_P1.27mm, F.Cu at (67.4, 79.4)
- added U134: 74LS244, Package_SO:SO-20_5.3x12.6mm_P1.27mm, F.Cu at (82.0, 79.4)
- added U135: 74LS32, Package_SO:SOIC-14_3.9x8.7mm_P1.27mm, F.Cu at (163.7, 35.2)
- added U91: 74ALS138, Package_SO:SOIC-16_3.9x9.9mm_P1.27mm, F.Cu at (-98.6, 11.1)
- added U92: 74LS374, Package_SO:SO-20_5.3x12.6mm_P1.27mm, F.Cu at (106.4, 62.8)
- added U95: 74LS244, Package_SO:SO-20_5.3x12.6mm_P1.27mm, F.Cu at (121.0, 62.9)
- added U99: 74LS374, Package_SO:SO-20_5.3x12.6mm_P1.27mm, F.Cu at (106.4, 79.4)
- U67: value 74LS138 -> 74ALS138
- moved U42 39.5 mm to (-41.0, 69.1)
- moved J3 28.2 mm to (22.4, 35.7)
- moved U70 28.2 mm to (82.6, 28.9)
- moved J2 28.2 mm to (22.4, -7.54)
- moved U72 28.2 mm to (48.4, -2.34)
- moved U73 28.2 mm to (48.4, 14.1)
- moved U74 28.2 mm to (82.6, -2.34)
- moved U71 28.2 mm to (58.1, 0.86)
- moved U75 28.2 mm to (82.6, 14.1)
- moved U77 28.2 mm to (37.4, 28.8)
- moved U82 28.2 mm to (48.4, 28.8)
- moved U98 27.3 mm to (155.3, 35.2)
- moved J28 5.34 mm to (99.1, 42.4)
- moved J29 5.34 mm to (128.3, 42.4)
- moved J30 5.34 mm to (113.8, 41.9)
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Connections:
- U110 pad 1: Net-(U116B-Q) -> unconnected-(U110-Pad1)
- U110 pad 2: Net-(U108-Pad12) -> unconnected-(U110-Pad2)
- U110 pad 3: /DragonInterface/latchData -> unconnected-(U110-Pad3)
- U25 pad 10: unconnected-(U25-Pad10) -> ~{ClkExtWrite}
- U25 pad 11: unconnected-(U25-Pad11) -> /ControlRegisters/~{RegisterRead5}
- U25 pad 12: unconnected-(U25-Pad12) -> /ControlRegisters/~{SelectRegister5}
- U25 pad 13: unconnected-(U25-Pad13) -> ~{ClkExtRead}
- U25 pad 8: unconnected-(U25-Pad8) -> /ControlRegisters/~{RegisterWrite5}
- U25 pad 9: unconnected-(U25-Pad9) -> /ControlRegisters/~{SelectRegister5}
- U67 pad 5: GND -> ~{RegBank0}
- U76 pad 10: /ControlRegisters/~{A1} -> unconnected-(U76-Pad10)
- U76 pad 11: /A1 -> unconnected-(U76-Pad11)
- U76 pad 3: /A0 -> unconnected-(U76-Pad3)
- U76 pad 4: /ControlRegisters/~{A0} -> unconnected-(U76-Pad4)
- U93 pad 10: ~{ExtWrite} -> ~{ClkExtWrite}
- U93 pad 13: ~{ExtRead} -> ~{ClkExtRead}
- U93 pad 2: ~{ExtWrite} -> ~{ClkExtWrite}
- U93 pad 5: ~{ExtRead} -> ~{ClkExtRead}
- U94 pad 10: ~{ExtWrite} -> ~{ClkExtWrite}
- U94 pad 13: ~{ExtRead} -> ~{ClkExtRead}
- U94 pad 2: ~{ExtWrite} -> ~{ClkExtWrite}
- U94 pad 5: ~{ExtRead} -> ~{ClkExtRead}
- U98 pad 10: GND -> ~{ClkExtWrite}
- U98 pad 11: unconnected-(U98-Pad11) -> /ControlRegisters/~{RegisterRead4}
- U98 pad 12: GND -> /ControlRegisters/~{SelectRegister4}
- U98 pad 13: GND -> ~{ClkExtRead}
- U98 pad 3: ~{ExtWrite} -> ~{ClkExtWrite}
- U98 pad 6: ~{ExtRead} -> ~{ClkExtRead}
- U98 pad 8: unconnected-(U98-Pad8) -> /ControlRegisters/~{RegisterWrite4}
- U98 pad 9: GND -> /ControlRegisters/~{SelectRegister4}
Routing:
- net /XD7: track 155.7 -> 306.7 mm, vias 8 -> 16
- net /XD6: track 135.3 -> 266.0 mm, vias 8 -> 16
- net /XD4: track 108.0 -> 211.4 mm, vias 4 -> 8
- net /XD5: track 105.3 -> 206.0 mm, vias 8 -> 16
- net /XD3: track 95.5 -> 151.0 mm
- net /XD2: track 89.8 -> 140.6 mm
- net /XD1: track 76.4 -> 114.6 mm
- net /XD0: track 70.1 -> 103.2 mm
- net /ControlRegisters/R5B7: track 0.00 -> 29.9 mm, vias 0 -> 4
- net /ControlRegisters/R4B7: track 0.00 -> 29.9 mm, vias 0 -> 4
- net /ControlRegisters/R7B7: track 0.00 -> 29.9 mm, vias 0 -> 4
- net /ControlRegisters/R6B7: track 0.00 -> 29.9 mm, vias 0 -> 4
- net /ControlRegisters/R4B4: track 0.00 -> 27.7 mm, vias 0 -> 1
- net /ControlRegisters/R6B4: track 0.00 -> 27.7 mm, vias 0 -> 1
- net /ControlRegisters/R5B4: track 0.00 -> 27.7 mm, vias 0 -> 1
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