File: DIY-Video.kicad_pcb (KiCad board)
At the start: 4 copper layers, 258.4 x 172.5 mm, 238 parts, among them IC26 MC6821, J1 VIDEO IO, J10 PosResets, J11 Power and Clock, J12 posX, J13 posY, J14 TimingTriggers, J15 ViewportOutput, J16 Power and Clock, J17 Triggers, J18 OpMode, J19 XDBus, J2 Host Address Bus, J20 XDBus, J21 Register0, J22 XDBus, J23 XDBus, J24 Register2, J25 XDBus, J26 XDBus, J27 Register1, J28 XDBus, J29 XDBus, J3 Host Data Bus, J30 Register3, J31 XDBus, J32 XDBus, J33 Register4, J34 XDBus, J35 XDBus, J36 Register6, J37 XDBus, J38 XDBus, J39 Register5, J4 Host Control Bus, J40 XDBus, J41 XDBus, J42 Register7, J5 posX, J6 posY, J7 ViewportTriggers, J8 posX, J9 posY, U1 74LS163, U10 74LS30, U100 74LS374, U101 74LS374, U102 74LS163, U103 74LS04, U104 74LS21, U105 74LS138, U106 74LS32, U107 74LS138, U108 74LS04, U109 74LS11, U11 74LS00, U110 74LS08, U111 74LS30, U112 74LS30, U113 74LS30, U114 74LS00, U115 74LS32, U116 74LS279, U117 74LS08, U118 74LS04, U119 74LS08, U12 74LS30, U120 74LS32, U121 74LS163, U122 74LS163, U123 74LS373, U124 74LS373, U125 74LS244, U126 74LS244, U127 74LS04, U128 74LS04, U129 74LS30, U13 74LS20, U130 74LS244, U131 74LS374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

Commit message: refine main board layout
Parts:
- added C1: 10nF, Capacitor_SMD:C_0603_1608Metric, F.Cu at (32.0, 112.0)
- added C10: 10nF, Capacitor_SMD:C_0603_1608Metric, F.Cu at (43.1, 139.4)
- added C11: 10nF, Capacitor_SMD:C_0603_1608Metric, F.Cu at (53.8, 139.6)
- added C12: 10nF, Capacitor_SMD:C_0603_1608Metric, F.Cu at (64.3, 139.3)
- added C13: 10nF, Capacitor_SMD:C_0603_1608Metric, F.Cu at (130.3, 104.6)
- added C14: 10nF, Capacitor_SMD:C_0603_1608Metric, F.Cu at (140.0, 104.6)
- added C15: 10nF, Capacitor_SMD:C_0603_1608Metric, F.Cu at (149.6, 104.6)
- added C16: 10nF, Capacitor_SMD:C_0603_1608Metric, F.Cu at (130.2, 115.4)
- added C17: 10nF, Capacitor_SMD:C_0603_1608Metric, F.Cu at (140.0, 115.4)
- added C18: 10nF, Capacitor_SMD:C_0603_1608Metric, F.Cu at (149.6, 115.4)
- added C19: 10nF, Capacitor_SMD:C_0603_1608Metric, F.Cu at (159.0, 115.4)
- added C2: 10nF, Capacitor_SMD:C_0603_1608Metric, F.Cu at (43.1, 111.9)
- added C20: 10nF, Capacitor_SMD:C_0603_1608Metric, F.Cu at (130.3, 126.2)
- added C21: 10nF, Capacitor_SMD:C_0603_1608Metric, F.Cu at (140.0, 126.2)
- added C22: 10nF, Capacitor_SMD:C_0603_1608Metric, F.Cu at (130.3, 137.1)
- added C23: 10nF, Capacitor_SMD:C_0603_1608Metric, F.Cu at (140.0, 137.1)
- added C24: 10nF, Capacitor_SMD:C_0603_1608Metric, F.Cu at (149.6, 137.1)
- added C25: 10nF, Capacitor_SMD:C_0603_1608Metric, F.Cu at (159.0, 137.1)
- added C26: 10nF, Capacitor_SMD:C_0603_1608Metric, F.Cu at (130.3, 149.5)
- added C27: 10nF, Capacitor_SMD:C_0603_1608Metric, F.Cu at (149.6, 149.5)
- added C3: 10nF, Capacitor_SMD:C_0603_1608Metric, F.Cu at (53.2, 112.0)
- added C4: 10nF, Capacitor_SMD:C_0603_1608Metric, F.Cu at (64.3, 111.9)
- added C5: 10nF, Capacitor_SMD:C_0603_1608Metric, F.Cu at (32.0, 125.7)
- added C6: 10nF, Capacitor_SMD:C_0603_1608Metric, F.Cu at (43.0, 125.6)
- added C7: 10nF, Capacitor_SMD:C_0603_1608Metric, F.Cu at (53.2, 125.6)
- added C8: 10nF, Capacitor_SMD:C_0603_1608Metric, F.Cu at (64.3, 125.6)
- added C9: 10nF, Capacitor_SMD:C_0603_1608Metric, F.Cu at (32.0, 139.4)
- added J43: Power, Connector_PinSocket_2.54mm:PinSocket_1x04_P2.54mm_Vertical, B.Cu at (167.7, 162.6)
- added J44: Power, Connector_PinSocket_2.54mm:PinSocket_1x04_P2.54mm_Vertical, B.Cu at (88.3, 170.2)
- added J45: Power and Clock, Connector_PinSocket_2.54mm:PinSocket_1x04_P2.54mm_Vertical, B.Cu at (104.4, 197.8)
- added J46: Triggers, Connector_PinSocket_2.54mm:PinSocket_1x04_P2.54mm_Vertical, B.Cu at (175.4, 198.2)
- added J47: OpMode, Connector_PinSocket_2.54mm:PinSocket_1x04_P2.54mm_Vertical, B.Cu at (143.2, 191.4)
- J2, J3: moved to B.Cu
- moved U104 161.6 mm to (35.2, 63.6)
- moved U105 161.6 mm to (35.2, 74.6)
- moved U106 161.6 mm to (43.6, 63.6)
- moved U103 147.3 mm to (43.9, 75.7)
- moved J12 129.9 mm to (25.4, 172.3)
- moved J13 129.9 mm to (25.4, 200.3)
- moved U100 129.4 mm to (55.0, 65.3)
- moved U101 129.4 mm to (65.5, 65.3)
- moved U102 129.4 mm to (54.0, 78.3)
- moved U30 129.1 mm to (227.7, 183.8)
- moved U31 129.1 mm to (191.7, 182.4)
- moved U32 129.1 mm to (200.1, 182.4)
- moved U33 129.1 mm to (208.6, 182.4)
- moved U34 129.1 mm to (217.0, 182.4)
- moved U35 129.1 mm to (191.7, 194.0)
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Routing:
- net /FrameTiming/X6: track 181.4 -> 253.5 mm
- net /FrameTiming/X5: track 161.0 -> 221.9 mm
- net /FrameTiming/Y5: track 162.8 -> 212.6 mm
- net /FrameTiming/X2: track 181.9 -> 230.6 mm
- net +5V: track 167.0 -> 215.5 mm
- net /FrameTiming/X3: track 153.3 -> 201.1 mm
- net /FrameTiming/X8: track 171.4 -> 217.5 mm
- net ~{Format}: track 64.1 -> 109.5 mm
- net /FrameTiming/X9: track 141.1 -> 186.4 mm
- net /FrameTiming/Y1: track 105.3 -> 149.5 mm
- net /FrameTiming/Y7: track 91.9 -> 131.3 mm
- net /FrameTiming/X1: track 71.8 -> 110.2 mm
- net /FrameTiming/Y6: track 83.8 -> 121.8 mm
- net /FrameTiming/Y3: track 66.8 -> 102.4 mm, vias 4 -> 3
- net /FrameTiming/X7: track 84.1 -> 119.5 mm
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Other:
- board size 258.4 x 172.5 mm -> 240.2 x 195.5 mm
- board text added: "Pixel Clock"

Commit message: tighten layout for final sizing
Parts:
- removed IC26: MC6821, Package_DIP:DIP-40_W15.24mm
- removed J19, J20, J22, J23, J25, J26, J28, J29, J31, J32, J34, J35, J37, J38, J40, J41: XDBus, Connector_PinHeader_1.27mm:PinHeader_1x08_P1.27mm_Vertical
- removed J21: Register0, Connector_PinHeader_1.27mm:PinHeader_1x10_P1.27mm_Vertical
- removed J24: Register2, Connector_PinHeader_1.27mm:PinHeader_1x10_P1.27mm_Vertical
- removed J27: Register1, Connector_PinHeader_1.27mm:PinHeader_1x10_P1.27mm_Vertical
- removed J30: Register3, Connector_PinHeader_1.27mm:PinHeader_1x10_P1.27mm_Vertical
- removed J33: Register4, Connector_PinHeader_1.27mm:PinHeader_1x10_P1.27mm_Vertical
- removed J36: Register6, Connector_PinHeader_1.27mm:PinHeader_1x10_P1.27mm_Vertical
- removed J39: Register5, Connector_PinHeader_1.27mm:PinHeader_1x10_P1.27mm_Vertical
- removed J42: Register7, Connector_PinHeader_1.27mm:PinHeader_1x10_P1.27mm_Vertical
- removed NT49: NetTie_2, NetTie:NetTie-2_SMD_Pad0.5mm
- removed U107: 74LS138, Package_SO:SOIC-16_3.9x9.9mm_P1.27mm
- removed U108: 74LS04, Package_SO:SO-14_3.9x8.65mm_P1.27mm
- removed U109: 74LS11, Package_SO:SO-14_3.9x8.65mm_P1.27mm
- removed U116: 74LS279, Package_SO:SOIC-16_3.9x9.9mm_P1.27mm
- removed U117: 74LS08, Package_SO:SO-14_3.9x8.65mm_P1.27mm
- removed U120, U93, U94, U98: 74LS32, Package_SO:SO-14_3.9x8.65mm_P1.27mm
- removed U121, U122: 74LS163, Package_SO:SOIC-16_3.9x9.9mm_P1.27mm
- removed U123, U124: 74LS373, Package_SO:SOIC-20W_7.5x12.8mm_P1.27mm
- removed U125, U126: 74LS244, Package_SO:SOIC-20W_7.5x12.8mm_P1.27mm
- removed U130, U132, U134, U85, U87, U89, U95, U97: 74LS244, Package_SO:SO-20_5.3x12.6mm_P1.27mm
- removed U131, U133, U84, U86, U88, U92, U96, U99: 74LS374, Package_SO:SO-20_5.3x12.6mm_P1.27mm
- removed U135: 74LS32, Package_SO:SOIC-14_3.9x8.7mm_P1.27mm
- removed U67: 74ALS138, Package_SO:SOIC-16_3.9x9.9mm_P1.27mm
- added C28: 10nF, Capacitor_SMD:C_0603_1608Metric, F.Cu at (122.0, 208.7)
- added C29: 10nF, Capacitor_SMD:C_0603_1608Metric, F.Cu at (135.5, 208.7)
- added C30: 10nF, Capacitor_SMD:C_0603_1608Metric, F.Cu at (148.9, 208.7)
- added C31: 10nF, Capacitor_SMD:C_0603_1608Metric, F.Cu at (162.3, 208.7)
- added C32: 10nF, Capacitor_SMD:C_0603_1608Metric, F.Cu at (175.7, 208.7)
- added C33: 10nF, Capacitor_SMD:C_0603_1608Metric, F.Cu at (122.0, 230.3)
- added C34: 10nF, Capacitor_SMD:C_0603_1608Metric, F.Cu at (135.4, 230.3)
- added C35: 10nF, Capacitor_SMD:C_0603_1608Metric, F.Cu at (148.8, 230.4)
- added C36: 10nF, Capacitor_SMD:C_0603_1608Metric, F.Cu at (162.2, 230.4)
- added C37: 10nF, Capacitor_SMD:C_0603_1608Metric, F.Cu at (175.6, 230.4)
- added C38: 10nF, Capacitor_SMD:C_0603_1608Metric, F.Cu at (201.5, 77.9)
- added C39: 10nF, Capacitor_SMD:C_0603_1608Metric, F.Cu at (221.7, 77.5)
- added C40: 10nF, Capacitor_SMD:C_0603_1608Metric, F.Cu at (231.2, 77.5)
- added C41: 10nF, Capacitor_SMD:C_0603_1608Metric, F.Cu at (240.8, 77.5)
- added C42: 10nF, Capacitor_SMD:C_0603_1608Metric, F.Cu at (250.4, 77.5)
- added C43: 10nF, Capacitor_SMD:C_0603_1608Metric, F.Cu at (195.2, 97.1)
- added C44: 10nF, Capacitor_SMD:C_0603_1608Metric, F.Cu at (230.5, 97.1)
- added C45: 10nF, Capacitor_SMD:C_0603_1608Metric, F.Cu at (219.3, 110.2)
- added C46: 10nF, Capacitor_SMD:C_0603_1608Metric, F.Cu at (230.5, 110.2)
- added C47: 10nF, Capacitor_SMD:C_0603_1608Metric, F.Cu at (202.2, 115.8)
- added C48: 10nF, Capacitor_SMD:C_0603_1608Metric, F.Cu at (230.5, 123.4)
- added C49: 10nF, Capacitor_SMD:C_0603_1608Metric, F.Cu at (247.0, 117.2)
- added C50: 10nF, Capacitor_SMD:C_0603_1608Metric, F.Cu at (258.5, 117.2)
- added C51: 10nF, Capacitor_SMD:C_0603_1608Metric, F.Cu at (42.7, 80.8)
- added C52: 10nF, Capacitor_SMD:C_0603_1608Metric, F.Cu at (58.0, 80.8)
- added C53: 10nF, Capacitor_SMD:C_0603_1608Metric, F.Cu at (82.7, 80.8)
- added C54: 10nF, Capacitor_SMD:C_0603_1608Metric, F.Cu at (94.4, 80.8)
- added C55: 10nF, Capacitor_SMD:C_0603_1608Metric, F.Cu at (42.6, 94.0)
- added C56: 10nF, Capacitor_SMD:C_0603_1608Metric, F.Cu at (58.0, 94.0)
- added C57: 10nF, Capacitor_SMD:C_0603_1608Metric, F.Cu at (70.0, 94.0)
- added C58: 10nF, Capacitor_SMD:C_0603_1608Metric, F.Cu at (94.4, 94.0)
- added C59: 10nF, Capacitor_SMD:C_0603_1608Metric, F.Cu at (82.7, 107.3)
- added C60: 10nF, Capacitor_SMD:C_0603_1608Metric, F.Cu at (94.4, 107.2)
- added C61: 10nF, Capacitor_SMD:C_0603_1608Metric, F.Cu at (94.4, 120.5)
- added C62: 10nF, Capacitor_SMD:C_0603_1608Metric, F.Cu at (128.0, 81.4)
- added C63: 10nF, Capacitor_SMD:C_0603_1608Metric, F.Cu at (145.3, 81.5)
- added C64: 10nF, Capacitor_SMD:C_0603_1608Metric, F.Cu at (161.7, 81.5)
- added C65: 10nF, Capacitor_SMD:C_0603_1608Metric, F.Cu at (123.6, 87.0)
- added C66: 10nF, Capacitor_SMD:C_0603_1608Metric, F.Cu at (128.7, 91.0)
- added C67: 10nF, Capacitor_SMD:C_0603_1608Metric, F.Cu at (164.1, 96.3)
- added C68: 10nF, Capacitor_SMD:C_0603_1608Metric, F.Cu at (123.5, 103.1)
- added C69: 10nF, Capacitor_SMD:C_0603_1608Metric, F.Cu at (122.7, 120.4)
- added C70: 10nF, Capacitor_SMD:C_0603_1608Metric, F.Cu at (175.4, 118.9)
- added C71: 4.7uF, Capacitor_SMD:CP_Elec_4x3, F.Cu at (169.6, 100.1)
- added J100: Triggers, Connector_PinSocket_2.54mm:PinSocket_1x04_P2.54mm_Vertical, F.Cu at (180.2, 212.2)
- added J101: OpMode, Connector_PinSocket_2.54mm:PinSocket_1x04_P2.54mm_Vertical, F.Cu at (148.0, 205.4)
- added J102: Power and Clock, Connector_PinSocket_2.54mm:PinSocket_1x04_P2.54mm_Vertical, F.Cu at (109.3, 211.8)
- added J103: Power and Clock, Connector_PinSocket_2.54mm:PinSocket_1x04_P2.54mm_Vertical, F.Cu at (109.3, 233.5)
- added J104: Triggers, Connector_PinSocket_2.54mm:PinSocket_1x04_P2.54mm_Vertical, F.Cu at (180.2, 233.9)
- added J105: OpMode, Connector_PinSocket_2.54mm:PinSocket_1x04_P2.54mm_Vertical, F.Cu at (148.0, 227.0)
- added J48: OpMode, Connector_PinSocket_2.54mm:PinSocket_1x04_P2.54mm_Vertical, B.Cu at (187.4, 79.2)
- added J49: Default Palette, Connector_PinSocket_2.54mm:PinSocket_1x04_P2.54mm_Vertical, B.Cu at (258.4, 109.2)
- added J50: Output Palette, Connector_PinSocket_2.54mm:PinSocket_1x04_P2.54mm_Vertical, B.Cu at (250.8, 135.4)
- added J51: Triggers, Connector_PinSocket_2.54mm:PinSocket_1x04_P2.54mm_Vertical, B.Cu at (206.6, 135.4)
- added J52: Power and Clock, Connector_PinSocket_2.54mm:PinSocket_1x04_P2.54mm_Vertical, B.Cu at (258.3, 79.2)
- added J53: BDBus, Connector_PinHeader_2.54mm:PinHeader_1x08_P2.54mm_Vertical, B.Cu at (187.4, 114.0)
- added J54: BDBus, Connector_PinHeader_2.54mm:PinHeader_1x08_P2.54mm_Vertical, B.Cu at (180.4, 114.0)
- added J55: Power, Connector_PinSocket_2.54mm:PinSocket_1x04_P2.54mm_Vertical, B.Cu at (180.4, 96.9)
- added J56: XDBus, Connector_PinHeader_2.54mm:PinHeader_1x08_P2.54mm_Vertical, B.Cu at (115.6, 77.4)
- added J57: BitmapAddress, Connector_PinHeader_2.54mm:PinHeader_1x16_P2.54mm_Vertical, B.Cu at (108.9, 77.4)
- added J58: BitmapAddress, Connector_PinHeader_2.54mm:PinHeader_1x16_P2.54mm_Vertical, B.Cu at (102.6, 77.4)
- added J59: Control, Connector_PinHeader_2.54mm:PinHeader_1x08_P2.54mm_Vertical, B.Cu at (109.7, 135.4)
- added J60: Power, Connector_PinSocket_2.54mm:PinSocket_1x04_P2.54mm_Vertical, B.Cu at (31.3, 127.8)
- added J61: RowCountControl, Connector_PinHeader_2.54mm:PinHeader_1x08_P2.54mm_Vertical, B.Cu at (74.5, 77.4)
- added J62: Triggers, Connector_PinSocket_2.54mm:PinSocket_1x04_P2.54mm_Vertical, B.Cu at (95.0, 135.4)
- added J63: Reg0, Connector_PinHeader_2.54mm:PinHeader_1x08_P2.54mm_Vertical, F.Cu at (136.7, 68.6)
- added J64: Reg1, Connector_PinHeader_2.54mm:PinHeader_1x08_P2.54mm_Vertical, F.Cu at (136.7, 71.1)
- added J65: Reg2, Connector_PinHeader_2.54mm:PinHeader_1x08_P2.54mm_Vertical, F.Cu at (169.7, 68.6)
- added J66: Reg3, Connector_PinHeader_2.54mm:PinHeader_1x08_P2.54mm_Vertical, F.Cu at (169.7, 71.1)
- added J67: Reg4, Connector_PinHeader_2.54mm:PinHeader_1x08_P2.54mm_Vertical, F.Cu at (203.0, 68.5)
- added J68: Reg5, Connector_PinHeader_2.54mm:PinHeader_1x08_P2.54mm_Vertical, F.Cu at (203.0, 71.0)
- added J69: Reg6, Connector_PinHeader_2.54mm:PinHeader_1x08_P2.54mm_Vertical, F.Cu at (236.0, 68.6)
- added J70: Reg7, Connector_PinHeader_2.54mm:PinHeader_1x08_P2.54mm_Vertical, F.Cu at (236.0, 71.1)
- added J71: BitmapAddress, Connector_PinHeader_2.54mm:PinHeader_1x16_P2.54mm_Vertical, F.Cu at (102.6, 77.4)
- added J72: RowCountControl, Connector_PinHeader_2.54mm:PinHeader_1x08_P2.54mm_Vertical, F.Cu at (74.5, 77.4)
- added J73: Triggers, Connector_PinSocket_2.54mm:PinSocket_1x04_P2.54mm_Vertical, F.Cu at (95.0, 135.4)
- added J74: Power, Connector_PinSocket_2.54mm:PinSocket_1x04_P2.54mm_Vertical, F.Cu at (31.3, 127.8)
- added J75: XDBus, Connector_PinHeader_2.54mm:PinHeader_1x08_P2.54mm_Vertical, F.Cu at (115.6, 77.4)
- added J76: BDBus, Connector_PinHeader_2.54mm:PinHeader_1x08_P2.54mm_Vertical, F.Cu at (180.5, 114.0)
- added J77: Power, Connector_PinSocket_2.54mm:PinSocket_1x04_P2.54mm_Vertical, F.Cu at (180.4, 96.9)
- added J78: BitmapAddress, Connector_PinHeader_2.54mm:PinHeader_1x16_P2.54mm_Vertical, F.Cu at (109.0, 77.4)
- added J79: BDBus, Connector_PinHeader_2.54mm:PinHeader_1x08_P2.54mm_Vertical, F.Cu at (187.4, 114.0)
- added J80: OpMode, Connector_PinSocket_2.54mm:PinSocket_1x04_P2.54mm_Vertical, F.Cu at (187.4, 79.2)
- added J81: Power and Clock, Connector_PinSocket_2.54mm:PinSocket_1x04_P2.54mm_Vertical, F.Cu at (258.3, 79.2)
- added J82: Default Palette, Connector_PinSocket_2.54mm:PinSocket_1x04_P2.54mm_Vertical, F.Cu at (258.4, 109.2)
- added J83: Output Palette, Connector_PinSocket_2.54mm:PinSocket_1x04_P2.54mm_Vertical, F.Cu at (250.8, 135.4)
- added J84: Host Address Bus, Connector_PinHeader_2.54mm:PinHeader_1x16_P2.54mm_Vertical, F.Cu at (142.4, 77.4)
- added J85: Triggers, Connector_PinSocket_2.54mm:PinSocket_1x04_P2.54mm_Vertical, F.Cu at (206.5, 135.4)
- added J86: Power and Clock, Connector_PinSocket_2.54mm:PinSocket_1x04_P2.54mm_Vertical, F.Cu at (38.9, 142.1)
- added J87: posX, Connector_PinSocket_2.54mm:PinSocket_1x10_P2.54mm_Vertical, F.Cu at (102.6, 143.1)
- added J88: posY, Connector_PinSocket_2.54mm:PinSocket_1x10_P2.54mm_Vertical, F.Cu at (102.5, 171.0)
- added J89: PosResets, Connector_PinSocket_2.54mm:PinSocket_1x04_P2.54mm_Vertical, F.Cu at (51.1, 199.9)
- added J90: posX, Connector_PinSocket_2.54mm:PinSocket_1x10_P2.54mm_Vertical, F.Cu at (109.7, 143.1)
- added J91: posY, Connector_PinSocket_2.54mm:PinSocket_1x10_P2.54mm_Vertical, F.Cu at (109.8, 171.0)
- added J92: Power, Connector_PinSocket_2.54mm:PinSocket_1x04_P2.54mm_Vertical, F.Cu at (172.6, 199.6)
- added J93: ViewportTriggers, Connector_PinSocket_2.54mm:PinSocket_1x06_P2.54mm_Vertical, F.Cu at (180.2, 154.5)
- added J94: Power, Connector_PinSocket_2.54mm:PinSocket_1x04_P2.54mm_Vertical, F.Cu at (94.5, 205.7)
- added J95: posX, Connector_PinSocket_2.54mm:PinSocket_1x10_P2.54mm_Vertical, F.Cu at (31.7, 207.9)
- added J96: posY, Connector_PinSocket_2.54mm:PinSocket_1x10_P2.54mm_Vertical, F.Cu at (31.7, 235.9)
- added J97: TimingTriggers, Connector_PinSocket_2.54mm:PinSocket_1x06_P2.54mm_Vertical, F.Cu at (48.4, 264.0)
- added J98: ViewportOutput, Connector_PinSocket_2.54mm:PinSocket_1x06_P2.54mm_Vertical, F.Cu at (102.1, 245.0)
- added J99: XDBus, Connector_PinHeader_2.54mm:PinHeader_1x08_P2.54mm_Vertical, F.Cu at (48.5, 30.4)
- added U136: 74LS04, Package_SO:SOIC-14_3.9x8.7mm_P1.27mm, F.Cu at (191.4, 102.3)
- added U137: 74LS08, Package_SO:SOIC-14_3.9x8.7mm_P1.27mm, F.Cu at (118.9, 125.6)
- J3: value Host Data Bus -> Host Address Bus; footprint Connector_PinHeader_2.54mm:PinHeader_1x08_P2.54mm_Vertical -> Connector_PinHeader_2.54mm:PinHeader_1x16_P2.54mm_Vertical; moved to F.Cu
- moved U61 288.8 mm to (198.8, 185.1), turned to 90 degrees
- moved U42 259.0 mm to (190.5, 185.1), turned to 90 degrees
- moved U91 164.7 mm to (58.3, 61.0)
- moved U83 143.3 mm to (67.7, 60.9)
- moved U25 134.1 mm to (87.6, 38.4)
- moved U39 134.1 mm to (246.6, 83.3)
- moved U76 124.9 mm to (96.1, 38.4)
- moved U90 124.5 mm to (113.0, 38.4)
- moved J4 121.4 mm to (35.5, 30.4)
- moved U38 112.5 mm to (237.0, 83.3)
- moved U37 112.3 mm to (227.5, 83.3)
- moved U36 112.1 mm to (217.9, 83.3)
- moved U32 98.8 mm to (197.7, 83.7)
- moved U41 94.6 mm to (254.8, 123.1)
- moved U40 93.2 mm to (243.2, 123.0)
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Connections:
- J3 pad 1: /XD0 -> /RegisterInterface/A0
- J3 pad 2: /XD1 -> /RegisterInterface/A1
- J3 pad 3: /XD2 -> /RegisterInterface/A2
- J3 pad 4: /XD3 -> /RegisterInterface/A3
- J3 pad 5: /XD4 -> /RegisterInterface/A4
- J3 pad 6: /XD5 -> /RegisterInterface/A5
- J3 pad 7: /XD6 -> /RegisterInterface/A6
- J3 pad 8: /XD7 -> /RegisterInterface/A7
- U103 pad 10: /BitmapPixelData/~{MR} -> unconnected-(U103-Pad10)
- U103 pad 11: ~{HCountEnable} -> unconnected-(U103-Pad11)
- U119 pad 1: (no net) -> unconnected-(U119-Pad1)
- U119 pad 2: (no net) -> unconnected-(U119-Pad2)
- U119 pad 3: (no net) -> unconnected-(U119-Pad3)
- U29 pad 3: /BitmapPixelCounter/PT3 -> /BitmapPixelCounter/PT0
- U29 pad 4: /BitmapPixelCounter/PT2 -> /BitmapPixelCounter/PT1
- U29 pad 5: /BitmapPixelCounter/PT1 -> /BitmapPixelCounter/PT2
- U29 pad 6: /BitmapPixelCounter/PT0 -> /BitmapPixelCounter/PT3
- U30 pad 12: /BitmapPixelData/D4 -> /BitmapPixelData/D7
- U30 pad 13: /BitmapMemory/BD4 -> /BitmapMemory/BD7
- U30 pad 14: /BitmapMemory/BD5 -> /BitmapMemory/BD4
- U30 pad 15: /BitmapPixelData/D5 -> /BitmapPixelData/D4
- U30 pad 16: /BitmapPixelData/D6 -> /BitmapPixelData/D3
- U30 pad 17: /BitmapMemory/BD6 -> /BitmapMemory/BD3
- U30 pad 18: /BitmapMemory/BD7 -> /BitmapMemory/BD1
- U30 pad 19: /BitmapPixelData/D7 -> /BitmapPixelData/D1
- U30 pad 4: /BitmapMemory/BD1 -> /BitmapMemory/BD2
- U30 pad 5: /BitmapPixelData/D1 -> /BitmapPixelData/D2
- U30 pad 6: /BitmapPixelData/D2 -> /BitmapPixelData/D5
- U30 pad 7: /BitmapMemory/BD2 -> /BitmapMemory/BD5
- U30 pad 8: /BitmapMemory/BD3 -> /BitmapMemory/BD6
- U30 pad 9: /BitmapPixelData/D3 -> /BitmapPixelData/D6
- U35 pad 6: /BitmapPixelData/BPP2Palette1 -> unconnected-(U35-~{Z}-Pad6)
- U40 pad 10: GND -> /BitmapPixelData/DefaultPalette1
- U40 pad 11: /BitmapPixelData/BPP2Palette2 -> /BitmapPixelData/BPP2Palette1
- U40 pad 12: /BitmapPixelData/BPP4Palette2 -> /BitmapPixelData/BPP4Palette1
- U40 pad 9: /BitmapPixelData/BMPalette2 -> /BitmapPixelData/BMPalette1
- U41 pad 10: GND -> /BitmapPixelData/DefaultPalette3
- U41 pad 11: /BitmapPixelData/BPP2Palette3 -> /BitmapPixelData/DefaultPalette3
- U41 pad 4: /BitmapPixelData/BPP4Palette1 -> /BitmapPixelData/BPP4Palette2
- U41 pad 5: /BitmapPixelData/BPP2Palette1 -> /BitmapPixelData/DefaultPalette2
- U41 pad 6: /BitmapPixelData/DefaultPalette1 -> /BitmapPixelData/DefaultPalette2
- U41 pad 7: /BitmapPixelData/BMPalette1 -> /BitmapPixelData/BMPalette2
- U71 pad 27: ~{WriteEnable} -> ~{ExtWrite}
- U72 pad 11: /A4 -> /A7
- U72 pad 12: /BitmapMemory/BA3 -> /BitmapMemory/BA5
- U72 pad 13: /A5 -> /A6
- U72 pad 14: /BitmapMemory/BA2 -> /BitmapMemory/BA3
- U72 pad 15: /A6 -> /A4
- U72 pad 16: /BitmapMemory/BA1 -> /BitmapMemory/BA2
- U72 pad 17: /A7 -> /A1
- U72 pad 3: /BitmapMemory/BA7 -> /BitmapMemory/BA1
- U72 pad 4: /A1 -> /A2
- U72 pad 5: /BitmapMemory/BA6 -> /BitmapMemory/BA4
- U72 pad 6: /A2 -> /A3
- U72 pad 7: /BitmapMemory/BA5 -> /BitmapMemory/BA6
- U72 pad 8: /A3 -> /A5
- U72 pad 9: /BitmapMemory/BA4 -> /BitmapMemory/BA7
- U73 pad 11: /A12 -> Page14
- U73 pad 12: /BitmapMemory/BA11 -> /BitmapMemory/BA13
- U73 pad 13: Page13 -> /A12
- U73 pad 14: /BitmapMemory/BA10 -> /BitmapMemory/BA11
- U73 pad 15: Page14 -> /A10
- U73 pad 5: /BitmapMemory/BA14 -> /BitmapMemory/BA10
- U73 pad 6: /A10 -> /A11
- U73 pad 7: /BitmapMemory/BA13 -> /BitmapMemory/BA12
- U73 pad 8: /A11 -> Page13
- U73 pad 9: /BitmapMemory/BA12 -> /BitmapMemory/BA14
- U74 pad 11: /BitmapAddressRegister/IBA4 -> /BitmapAddressRegister/IBA7
- U74 pad 12: /BitmapMemory/BA3 -> /BitmapMemory/BA6
- U74 pad 14: /BitmapMemory/BA2 -> /BitmapMemory/BA4
- U74 pad 15: /BitmapAddressRegister/IBA6 -> /BitmapAddressRegister/IBA3
- U74 pad 16: /BitmapMemory/BA1 -> /BitmapMemory/BA2
- U74 pad 17: /BitmapAddressRegister/IBA7 -> /BitmapAddressRegister/IBA1
- U74 pad 3: /BitmapMemory/BA7 -> /BitmapMemory/BA1
- U74 pad 4: /BitmapAddressRegister/IBA1 -> /BitmapAddressRegister/IBA2
- U74 pad 5: /BitmapMemory/BA6 -> /BitmapMemory/BA3
- U74 pad 6: /BitmapAddressRegister/IBA2 -> /BitmapAddressRegister/IBA4
- U74 pad 8: /BitmapAddressRegister/IBA3 -> /BitmapAddressRegister/IBA6
- U74 pad 9: /BitmapMemory/BA4 -> /BitmapMemory/BA7
- U75 pad 11: /BitmapAddressRegister/IBA12 -> /BitmapAddressRegister/IBA13
- U75 pad 12: /BitmapMemory/BA11 -> /BitmapMemory/BA14
- U75 pad 13: /BitmapAddressRegister/IBA13 -> /BitmapAddressRegister/IBA11
- U75 pad 14: /BitmapMemory/BA10 -> /BitmapMemory/BA12
- U75 pad 15: /BitmapAddressRegister/IBA14 -> /BitmapAddressRegister/IBA9
- U75 pad 16: /BitmapMemory/BA9 -> /BitmapMemory/BA10
- U75 pad 4: /BitmapAddressRegister/IBA9 -> /BitmapAddressRegister/IBA10
- U75 pad 5: /BitmapMemory/BA14 -> /BitmapMemory/BA9
- U75 pad 6: /BitmapAddressRegister/IBA10 -> /BitmapAddressRegister/IBA12
- U75 pad 7: /BitmapMemory/BA13 -> /BitmapMemory/BA11
- U75 pad 8: /BitmapAddressRegister/IBA11 -> /BitmapAddressRegister/IBA14
- U75 pad 9: /BitmapMemory/BA12 -> /BitmapMemory/BA13
- U77 pad 11: /XD4 -> /XD6
- U77 pad 12: /BitmapMemory/D3 -> /BitmapMemory/D7
- U77 pad 13: /XD5 -> /XD4
- U77 pad 14: /BitmapMemory/D2 -> /BitmapMemory/D5
- U77 pad 15: /XD6 -> /XD2
- U77 pad 16: /BitmapMemory/D1 -> /BitmapMemory/D3
- U77 pad 17: /XD7 -> /XD0
- U77 pad 18: /BitmapMemory/D0 -> /BitmapMemory/D1
- U77 pad 2: /XD0 -> /XD1
- U77 pad 3: /BitmapMemory/D7 -> /BitmapMemory/D0
- U77 pad 4: /XD1 -> /XD3
- U77 pad 5: /BitmapMemory/D6 -> /BitmapMemory/D2
- U77 pad 6: /XD2 -> /XD5
- U77 pad 7: /BitmapMemory/D5 -> /BitmapMemory/D4
- U77 pad 8: /XD3 -> /XD7
- U77 pad 9: /BitmapMemory/D4 -> /BitmapMemory/D6
- U82 pad 11: /BitmapMemory/D4 -> /BitmapMemory/D6
- U82 pad 12: /XD3 -> /XD7
- U82 pad 13: /BitmapMemory/D5 -> /BitmapMemory/D4
- U82 pad 14: /XD2 -> /XD5
- U82 pad 15: /BitmapMemory/D6 -> /BitmapMemory/D2
- U82 pad 16: /XD1 -> /XD3
- U82 pad 17: /BitmapMemory/D7 -> /BitmapMemory/D0
- U82 pad 18: /XD0 -> /XD1
- U82 pad 2: /BitmapMemory/D0 -> /BitmapMemory/D1
- U82 pad 3: /XD7 -> /XD0
- U82 pad 4: /BitmapMemory/D1 -> /BitmapMemory/D3
- U82 pad 5: /XD6 -> /XD2
- U82 pad 6: /BitmapMemory/D2 -> /BitmapMemory/D5
- U82 pad 7: /XD5 -> /XD4
- U82 pad 8: /BitmapMemory/D3 -> /BitmapMemory/D7
- U82 pad 9: /XD4 -> /XD6
- U83 pad 1: /ControlRegisters/~{PageSize0} -> unconnected-(U83-Pad1)
- U83 pad 2: /A13 -> unconnected-(U83-Pad2)
- U83 pad 3: Net-(U25-Pad1) -> unconnected-(U83-Pad3)
- U90 pad 1: unconnected-(U90-Pad1) -> /ControlRegisters/~{PageSize0}
- U90 pad 2: unconnected-(U90-Pad2) -> /A13
- U90 pad 3: unconnected-(U90-Pad3) -> Net-(U25-Pad1)
Routing:
- net /XD7: track 331.1 -> 28.2 mm, vias 18 -> 2
- net /XD6: track 290.4 -> 23.2 mm, vias 18 -> 0
- net /XD4: track 233.5 -> 25.3 mm, vias 8 -> 0
- net /XD5: track 229.9 -> 30.4 mm, vias 18 -> 2
- net ~{HSync}: track 69.7 -> 220.1 mm, vias 2 -> 6
- net /BitmapAddressRegister/~{RRMR}: track 0.00 -> 150.1 mm, vias 0 -> 5
- net /BitmapPixelData/D3: track 0.00 -> 144.3 mm, vias 0 -> 4
- net GND: track 267.9 -> 408.8 mm, vias 197 -> 273
- net /BitmapPixelData/D7: track 0.00 -> 135.9 mm, vias 0 -> 4
- net PixelClock: track 0.00 -> 134.3 mm, vias 0 -> 4
- net /BitmapDataCounter/BPP0: track 42.4 -> 173.8 mm, vias 1 -> 2
- net /BitmapPixelData/D2: track 0.00 -> 130.6 mm, vias 0 -> 4
- net /BitmapDataCounter/BPP1: track 30.2 -> 160.1 mm
- net ~{BitmapRead}: track 0.00 -> 129.5 mm, vias 0 -> 4
- net ~{HCountEnable}: track 59.4 -> 181.8 mm, vias 0 -> 1
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Other:
- board size 240.2 x 195.5 mm -> 236.8 x 240.9 mm
- board text added: "Pixel Clock Divider"
- board text added: "Pixel Load Clock Divider"
- board text added: "Reserved for register controlled palette definition (Requires two control blocks)"
- board text removed: "Pixel Clock"
- board text removed: "Pixel Divider"
