File: AddressReguster.kicad_sch (KiCad schematic)
At the start: 11 parts, among them U100 74LS374, U101 74LS374, U102 74LS163, U103 74LS04, U104 74LS21, U105 74LS138, U106 74LS32, U78 74LS163, U79 74LS163, U80 74LS163, U81 74LS163

Commit message: fix x/y counters to reset at the correct positions
Parts:
- removed unit 4 of U103
Connections:
- no-connect marks 14 -> 13
Changed lines of the file:
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@@
 	)
 	(no_connect
-		(at 317.5 125.73)
-	)
-	(no_connect
 		(at 96.52 96.52)
 	)
@@
 					(unit 1)
 				)
-			)
-		)
-	)
-	(symbol
-		(lib_id "74xx:74LS04")
-		(at 309.88 125.73 0)
-		(unit 4)
-		(exclude_from_sim no)
-		(in_bom yes)
-		(on_board yes)
-		(dnp no)
-		(fields_autoplaced yes)
-		(property "Reference" "U103"
-			(at 309.88 116.84 0)
-			(effects
-				(font
-					(size 1.27 1.27)
-				)
-			)
-		)
-		(property "Value" "74LS04"
-			(at 309.88 119.38 0)
-			(effects
-				(font
-					(size 1.27 1.27)
-				)
-			)
-		)
-		(property "Footprint" ""
-			(at 309.88 125.73 0)
-			(effects
-				(font
-					(size 1.27 1.27)
-				)
-				(hide yes)
-			)
-		)
-		(property "Datasheet" "http://www.ti.com/lit/gpn/sn74LS04"
-			(at 309.88 125.73 0)
-			(effects
-				(font
-					(size 1.27 1.27)
-				)
-				(hide yes)
-			)
-		)
-		(property "Description" "Hex Inverter"
-			(at 309.88 125.73 0)
-			(effects
-				(font
-					(size 1.27 1.27)
-				)
-				(hide yes)
-			)
-		)
-		(pin "2"
-		)
-		(pin "1"
-		)
-		(pin "3"
-		)
-		(pin "4"
-		)
-		(pin "9"
-		)
-		(pin "5"
-		)
-		(pin "8"
-		)
-		(pin "11"
-		)
-		(pin "6"
-		)
-		(pin "10"
-		)
-		(pin "13"
-		)
-		(pin "12"
-		)
-		(pin "14"
-		)
-		(pin "7"
-		)
-		(instances
-			(project "DIY-Video"
-				(path "/6c4ef05c-ecf5-4bee-ae4e-d72f13738678/2dbadac2-cca2-450a-9e58-4b03ae55b963"
-					(reference "U103")
-					(unit 4)
-				)
-			)
-		)
-	)
-	(symbol
-		(lib_id "power:+5V")
-		(at 302.26 125.73 0)
-		(unit 1)
-		(exclude_from_sim no)
-		(in_bom yes)
-		(on_board yes)
-		(dnp no)
-		(fields_autoplaced yes)
-		(property "Reference" "#PWR0358"
-			(at 302.26 129.54 0)
-			(effects
-				(font
-					(size 1.27 1.27)
-				)
-				(hide yes)
-			)
-		)
-		(property "Value" "+5V"
-			(at 302.26 120.65 0)
-			(effects
-				(font
-					(size 1.27 1.27)
-				)
-			)
-		)
-		(property "Footprint" ""
-			(at 302.26 125.73 0)
-			(effects
-				(font
-					(size 1.27 1.27)
-				)
-				(hide yes)
-			)
-		)
-		(property "Datasheet" ""
-			(at 302.26 125.73 0)
-			(effects
-				(font
-					(size 1.27 1.27)
-				)
-				(hide yes)
-			)
-		)
-		(property "Description" "Power symbol creates a global label with name \"+5V\""
-			(at 302.26 125.73 0)
-			(effects
-				(font
-					(size 1.27 1.27)
-				)
-				(hide yes)
-			)
-		)
-		(pin "1"
-		)
-		(instances
-			(project "DIY-Video"
-				(path "/6c4ef05c-ecf5-4bee-ae4e-d72f13738678/2dbadac2-cca2-450a-9e58-4b03ae55b963"
-					(reference "#PWR0358")
-					(unit 1)
-				)

Commit message: test (and fix) BitmapPixelData
Parts:
- removed unit 5 of U103
Connections:
- no-connect marks 13 -> 12
Changed lines of the file:
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@@
 	)
 	(no_connect
-		(at 317.5 139.7)
-	)
-	(no_connect
 		(at 139.7 101.6)
 	)
@@
 	)
 	(symbol
-		(lib_id "74xx:74LS04")
-		(at 309.88 139.7 0)
-		(unit 5)
-		(exclude_from_sim no)
-		(in_bom yes)
-		(on_board yes)
-		(dnp no)
-		(fields_autoplaced yes)
-		(property "Reference" "U103"
-			(at 309.88 130.81 0)
-			(effects
-				(font
-					(size 1.27 1.27)
-				)
-			)
-		)
-		(property "Value" "74LS04"
-			(at 309.88 133.35 0)
-			(effects
-				(font
-					(size 1.27 1.27)
-				)
-			)
-		)
-		(property "Footprint" ""
-			(at 309.88 139.7 0)
-			(effects
-				(font
-					(size 1.27 1.27)
-				)
-				(hide yes)
-			)
-		)
-		(property "Datasheet" "http://www.ti.com/lit/gpn/sn74LS04"
-			(at 309.88 139.7 0)
-			(effects
-				(font
-					(size 1.27 1.27)
-				)
-				(hide yes)
-			)
-		)
-		(property "Description" "Hex Inverter"
-			(at 309.88 139.7 0)
-			(effects
-				(font
-					(size 1.27 1.27)
-				)
-				(hide yes)
-			)
-		)
-		(pin "2"
-		)
-		(pin "1"
-		)
-		(pin "3"
-		)
-		(pin "4"
-		)
-		(pin "9"
-		)
-		(pin "5"
-		)
-		(pin "8"
-		)
-		(pin "11"
-		)
-		(pin "6"
-		)
-		(pin "10"
-		)
-		(pin "13"
-		)
-		(pin "12"
-		)
-		(pin "14"
-		)
-		(pin "7"
-		)
-		(instances
-			(project "DIY-Video"
-				(path "/6c4ef05c-ecf5-4bee-ae4e-d72f13738678/2dbadac2-cca2-450a-9e58-4b03ae55b963"
-					(reference "U103")
-					(unit 5)
-				)
-			)
-		)
-	)
-	(symbol
 		(lib_id "power:GND")
 		(at 39.37 175.26 0)
@@
 					(unit 1)
 				)
-			)
-		)
-	)
-	(symbol
-		(lib_id "power:+5V")
-		(at 302.26 139.7 0)
-		(unit 1)
-		(exclude_from_sim no)
-		(in_bom yes)
-		(on_board yes)
-		(dnp no)
-		(fields_autoplaced yes)
-		(property "Reference" "#PWR0355"
-			(at 302.26 143.51 0)
-			(effects
-				(font
-					(size 1.27 1.27)
-				)
-				(hide yes)
-			)
-		)
-		(property "Value" "+5V"
-			(at 302.26 134.62 0)
-			(effects
-				(font
-					(size 1.27 1.27)
-				)
-			)
-		)
-		(property "Footprint" ""
-			(at 302.26 139.7 0)
-			(effects
-				(font
-					(size 1.27 1.27)
-				)
-				(hide yes)
-			)
-		)
-		(property "Datasheet" ""
-			(at 302.26 139.7 0)
-			(effects
-				(font
-					(size 1.27 1.27)
-				)
-				(hide yes)
-			)
-		)
-		(property "Description" "Power symbol creates a global label with name \"+5V\""
-			(at 302.26 139.7 0)
-			(effects
-				(font
-					(size 1.27 1.27)
-				)
-				(hide yes)
-			)
-		)
-		(pin "1"
-		)
-		(instances
-			(project "DIY-Video"
-				(path "/6c4ef05c-ecf5-4bee-ae4e-d72f13738678/2dbadac2-cca2-450a-9e58-4b03ae55b963"
-					(reference "#PWR0355")
-					(unit 1)
-				)

Commit message: spin register out as separate board
Parts:
- U103, U104, U106: footprint (none) -> Package_SO:SOIC-14_3.9x8.7mm_P1.27mm
- U105: footprint (none) -> Package_SO:SOIC-16_3.9x9.9mm_P1.27mm
Changed lines of the file:
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@@
 			)
 		)
-		(property "Footprint" ""
+		(property "Footprint" "Package_SO:SOIC-14_3.9x8.7mm_P1.27mm"
 			(at 309.88 167.64 0)
 			(effects
@@
 			)
 		)
-		(property "Footprint" ""
+		(property "Footprint" "Package_SO:SOIC-14_3.9x8.7mm_P1.27mm"
 			(at 254 102.87 0)
 			(effects
@@
 			)
 		)
-		(property "Footprint" ""
+		(property "Footprint" "Package_SO:SOIC-14_3.9x8.7mm_P1.27mm"
 			(at 111.76 166.37 0)
 			(effects
@@
 			)
 		)
-		(property "Footprint" ""
+		(property "Footprint" "Package_SO:SOIC-14_3.9x8.7mm_P1.27mm"
 			(at 127 153.67 0)
 			(effects
@@
 			)
 		)
-		(property "Footprint" ""
+		(property "Footprint" "Package_SO:SOIC-14_3.9x8.7mm_P1.27mm"
 			(at 234.95 102.87 0)
 			(effects
@@
 			)
 		)
-		(property "Footprint" ""
+		(property "Footprint" "Package_SO:SOIC-14_3.9x8.7mm_P1.27mm"
 			(at 309.88 153.67 0)
 			(effects
@@
 			)
 		)
-		(property "Footprint" ""
+		(property "Footprint" "Package_SO:SOIC-14_3.9x8.7mm_P1.27mm"
 			(at 127 143.51 0)
 			(effects
@@
 			)
 		)
-		(property "Footprint" ""
+		(property "Footprint" "Package_SO:SOIC-14_3.9x8.7mm_P1.27mm"
 			(at 158.75 144.78 0)
 			(effects
@@
 			)
 		)
-		(property "Footprint" ""
+		(property "Footprint" "Package_SO:SOIC-14_3.9x8.7mm_P1.27mm"
 			(at 111.76 156.21 0)
 			(effects
@@
 			)
 		)
-		(property "Footprint" ""
+		(property "Footprint" "Package_SO:SOIC-14_3.9x8.7mm_P1.27mm"
 			(at 116.84 184.15 0)
 			(effects
@@
 			)
 		)
-		(property "Footprint" ""
+		(property "Footprint" "Package_SO:SOIC-14_3.9x8.7mm_P1.27mm"
 			(at 127 163.83 0)
 			(effects
@@
 			)
 		)
-		(property "Footprint" ""
+		(property "Footprint" "Package_SO:SOIC-16_3.9x9.9mm_P1.27mm"
 			(at 83.82 153.67 0)
 			(effects
@@
 			)
 		)
-		(property "Footprint" ""
+		(property "Footprint" "Package_SO:SOIC-14_3.9x8.7mm_P1.27mm"
 			(at 111.76 146.05 0)
 			(effects
@@
 			)
 		)
-		(property "Footprint" ""
+		(property "Footprint" "Package_SO:SOIC-14_3.9x8.7mm_P1.27mm"
 			(at 215.9 102.87 0)
 			(effects

Commit message: tighten layout for final sizing
Parts:
- added C51, C52, C53, C54, C55, C56, C57, C58, C59, C60, C61: 10nF, Capacitor_SMD:C_0603_1608Metric, symbol Device:C_Small
- added J57: BitmapAddress, Connector_PinHeader_2.54mm:PinHeader_1x16_P2.54mm_Vertical, symbol Connector_Generic:Conn_01x16
- added J60: Power, Connector_PinSocket_2.54mm:PinSocket_1x04_P2.54mm_Vertical, symbol Connector_Generic:Conn_01x04
- added J61: RowCountControl, Connector_PinHeader_2.54mm:PinHeader_1x08_P2.54mm_Vertical, symbol Connector_Generic:Conn_01x08
- added J62: Triggers, Connector_PinSocket_2.54mm:PinSocket_1x04_P2.54mm_Vertical, symbol Connector_Generic:Conn_01x04
- added unit 5 of U103
Connections:
- net +5V: now also C51.1, C52.1, C53.1, C54.1, C55.1, C56.1, C57.1, C58.1, C59.1, C60.1, C61.1, J60.1 (Pin_1), J60.4 (Pin_4)
- net GND: now also C51.2, C52.2, C53.2, C54.2, C55.2, C56.2, C57.2, C58.2, C59.2, C60.2, C61.2, J60.2 (Pin_2), J60.3 (Pin_3)
- net IBA0: now also J57.1 (Pin_1)
- net IBA1: now also J57.2 (Pin_2)
- net IBA10: now also J57.11 (Pin_11)
- net IBA11: now also J57.12 (Pin_12)
- net IBA12: now also J57.13 (Pin_13)
- net IBA13: now also J57.14 (Pin_14)
- net IBA14: now also J57.15 (Pin_15)
- net IBA2: now also J57.3 (Pin_3)
- net IBA3: now also J57.4 (Pin_4)
- net IBA4: now also J57.5 (Pin_5)
- net IBA5: now also J57.6 (Pin_6)
- net IBA6: now also J57.7 (Pin_7)
- net IBA7: now also J57.8 (Pin_8)
- net IBA8: now also J57.9 (Pin_9)
- net IBA9: now also J57.10 (Pin_10)
- net RC0: now also J61.2 (Pin_2)
- net RC1: now also J61.3 (Pin_3)
- net RC2: now also J61.4 (Pin_4)
- net RC3: now also J61.5 (Pin_5)
- net RR0: now also J61.6 (Pin_6)
- net RR1: now also J61.7 (Pin_7)
- net ~{HLoad}: now also J62.1 (Pin_1)
- net ~{HSync}: now also J62.2 (Pin_2)
- net ~{RRMR}: now also J61.1 (Pin_1)
- net ~{VSync}: now also J62.3 (Pin_3)
- no-connect marks 12 -> 15
