File: BitmaPixelData.kicad_sch (KiCad schematic)
At the start: 12 parts, among them U30 74LS373, U31 74LS163, U32 74LS138, U33 74LS151, U34 74LS151, U35 74LS151, U36 74LS151, U37 74LS151, U38 74LS151, U39 74LS151, U40 74LS352, U41 74LS352

Commit message: provide annotation on modules
Changed lines of the file:
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@@
+		)
+	)
+	(text_box "The process of selecting the relevant bits from the data register is performed by using a group of multiplexers.\n\nFor 1 BPP a single multiplexer is used. For 2 BPP two multiplexers are needed, selecting alternate bits on each count but out of phase.\n\nFor 4 BPP the system needs four multiplexers, selecting the 1st, 2nd, 3rd and 4th bit, or the 5th, 6th, 7th and 8th bit"
+		(exclude_from_sim no)
+		(at 175.26 139.7 0)
+		(size 48.26 24.13)
+		(margins 0.9525 0.9525 0.9525 0.9525)
+		(stroke
+			(width 0)
+			(type solid)
+		)
+		(fill
+			(type color)
+			(color 255 255 255 1)
+		)
+		(effects
+			(font
+				(size 1.27 1.27)
+			)
+			(justify left top)
+		)
+	)
+	(text_box "The BitmapPixelData module is technically 3 modules in one. Each is responsible for defining the palette index from the current bitmap data\n\nTraditionally the bitmap data would be held in a shift register, rotated out with each pixel transition.\n\nDue to the variable bitmap data length the system uses a multiplexing mechanism to switch between bit positions with an effective data length of 1, 2 or 4 bits. This saves on triggering a variable number of clock pulses to shift sufficient data out of the register holding the bitmap data\n\nThe final element in this is pulling the unused bits of the palette index to 0 so that the lowest 2 or 4 indexes are used. This could be substituted with a control register held value that changes which consecutive sequence is utilised. It still limits the effective palette to a fixed selection but does offer some additional control. This would be more effective if the palette is programmable but in that event the need to use anything more than the lowest palette options is largely negated"
+		(exclude_from_sim no)
+		(at 124.46 139.7 0)
+		(size 50.8 57.15)
+		(margins 0.9525 0.9525 0.9525 0.9525)
+		(stroke
+			(width 0)
+			(type solid)
+		)
+		(fill
+			(type color)
+			(color 255 255 255 1)
+		)
+		(effects
+			(font
+				(size 1.27 1.27)
+			)
+			(justify left top)
 		)
 	)
@@
 	)
 	(bus_entry
-		(at 140.97 157.48)
+		(at 264.16 148.59)
 		(size 2.54 2.54)
 		(stroke
@@
 	)
 	(bus_entry
-		(at 140.97 162.56)
+		(at 264.16 153.67)
 		(size 2.54 2.54)
 		(stroke
@@
 	)
 	(bus_entry
-		(at 140.97 160.02)
+		(at 264.16 151.13)
 		(size 2.54 2.54)
 		(stroke
@@
 	)
 	(bus_entry
-		(at 140.97 165.1)
+		(at 264.16 156.21)
 		(size 2.54 2.54)
 		(stroke
@@
 	(wire
 		(pts
-			(xy 143.51 167.64) (xy 144.78 167.64)
+			(xy 266.7 158.75) (xy 267.97 158.75)
 		)
 		(stroke
@@
 	(wire
 		(pts
-			(xy 143.51 160.02) (xy 144.78 160.02)
+			(xy 266.7 151.13) (xy 267.97 151.13)
 		)
 		(stroke
@@
 	(bus
 		(pts
-			(xy 140.97 157.48) (xy 140.97 160.02)
+			(xy 264.16 148.59) (xy 264.16 151.13)
 		)
 		(stroke
@@
 	(wire
 		(pts
-			(xy 143.51 162.56) (xy 144.78 162.56)
+			(xy 266.7 153.67) (xy 267.97 153.67)
 		)
 		(stroke
@@
 	(bus
 		(pts
-			(xy 140.97 162.56) (xy 140.97 165.1)
+			(xy 264.16 153.67) (xy 264.16 156.21)
 		)
 		(stroke
@@
 	(wire
 		(pts
-			(xy 143.51 165.1) (xy 144.78 165.1)
+			(xy 266.7 156.21) (xy 267.97 156.21)
 		)
 		(stroke
@@
 	(bus
 		(pts
-			(xy 140.97 160.02) (xy 140.97 162.56)
+			(xy 264.16 151.13) (xy 264.16 153.67)
 		)
 		(stroke
@@
 	(bus
 		(pts
-			(xy 140.97 154.94) (xy 140.97 157.48)
+			(xy 264.16 146.05) (xy 264.16 148.59)
 		)
 		(stroke
@@
 	)
 	(label "BMPalette1"
-		(at 144.78 162.56 0)
+		(at 267.97 153.67 0)
 		(effects
 			(font
@@
 	)
 	(label "BMPalette2"
-		(at 144.78 165.1 0)
+		(at 267.97 156.21 0)
 		(effects
 			(font
@@
 	)
 	(label "BMPalette0"
-		(at 144.78 160.02 0)
+		(at 267.97 151.13 0)
 		(effects
 			(font
@@
 	)
 	(label "BMPalette3"
-		(at 144.78 167.64 0)
+		(at 267.97 158.75 0)
 		(effects
 			(font
@@
 	(hierarchical_label "BMPalette[0..3]"
 		(shape output)
-		(at 140.97 154.94 0)
-		(effects
-			(font
+		(at 264.16 146.05 0)
+		(effects
+			(font

Commit message: test (and fix) BitmapPixelData
Parts:
- removed U40, U41: 74LS352, Package_SO:SOIC-16_3.9x9.9mm_P1.27mm, symbol 74xx:74LS352
- added U103: 74LS04, symbol 74xx:74LS04
- added U40, U41: 74LS153, symbol 74xx:74LS153
Connections:
- net +5V: now also U31.1 (~{MR}), U31.3 (D0), U31.4 (D1), U31.5 (D2), U31.6 (D3), U40.16 (VCC), U41.16 (VCC)
- net BMPalette0: now also U40.7 (Za)
- net BMPalette1: now also U41.7 (Za)
- net BMPalette2: now also U40.9 (Zb)
- net BMPalette3: now also U41.9 (Zb)
- net BPP0: now also U40.14 (S0), U41.14 (S0)
- net BPP1: now also U40.2 (S1), U41.2 (S1)
- net BPP1Palette0: now also U40.6 (I0a)
- net BPP2Palette0: now also U40.5 (I1a)
- net BPP2Palette1: now also U41.5 (I1a)
- net BPP2Palette2: now also U40.11 (I1b)
- net BPP2Palette3: now also U41.11 (I1b)
- net BPP4Palette0: now also U40.4 (I2a)
- net BPP4Palette1: now also U41.4 (I2a)
- net BPP4Palette2: now also U40.12 (I2b)
- net BPP4Palette3: now also U41.12 (I2b)
- net D0: now also U33.12 (I7), U34.1 (I3), U36.3 (I1); no longer U33.4 (I0), U34.4 (I0), U36.4 (I0)
- net D1: now also U33.13 (I6), U35.1 (I3), U37.3 (I1); no longer U33.3 (I1), U35.4 (I0), U37.4 (I0)
- net D2: now also U33.14 (I5), U34.2 (I2), U38.3 (I1); no longer U33.2 (I2), U34.3 (I1), U38.4 (I0)
- net D3: now also U33.15 (I4), U35.2 (I2), U39.3 (I1); no longer U33.1 (I3), U35.3 (I1), U39.4 (I0)
- net D4: now also U33.1 (I3), U34.3 (I1), U36.4 (I0); no longer U33.15 (I4), U34.2 (I2), U36.3 (I1)
- net D5: now also U33.2 (I2), U35.3 (I1), U37.4 (I0); no longer U33.14 (I5), U35.2 (I2), U37.3 (I1)
- net D6: now also U33.3 (I1), U34.4 (I0), U38.4 (I0); no longer U33.13 (I6), U34.1 (I3), U38.3 (I1)
- net D7: now also U33.4 (I0), U35.4 (I0), U39.4 (I0); no longer U33.12 (I7), U35.1 (I3), U39.3 (I1)
- net GND: now also U40.1 (Ea), U40.10 (I0b), U40.13 (I3b), U40.15 (Eb), U40.3 (I3a), U40.8 (GND), U41.1 (Ea), U41.10 (I0b), U41.13 (I3b), U41.15 (Eb), U41.3 (I3a), U41.8 (GND); no longer U31.1 (~{MR}), U31.3 (D0), U31.4 (D1), U31.5 (D2), U31.6 (D3), U31.9 (~{PE})
- new net BPP1Palette1: U41.6 (I0a)
- new net ~{HCountEnable}: U103.11
- new net ~{MR}: U103.10, U31.9 (~{PE})
Other:
- note added: "Counter reset needs to go to $F not $0 to avoid skipping the first pixel"
- moved on the sheet: U31, U32

Commit message: spin register out as separate board
Parts:
- U103: footprint (none) -> Package_SO:SOIC-14_3.9x8.7mm_P1.27mm
- U40, U41: footprint (none) -> Package_SO:SOIC-16_3.9x9.9mm_P1.27mm
Changed lines of the file:
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@@
 			)
 		)
-		(property "Footprint" ""
+		(property "Footprint" "Package_SO:SOIC-16_3.9x9.9mm_P1.27mm"
 			(at 43.18 162.56 0)
 			(effects
@@
 			)
 		)
-		(property "Footprint" ""
+		(property "Footprint" "Package_SO:SOIC-14_3.9x8.7mm_P1.27mm"
 			(at 36.83 64.77 0)
 			(effects
@@
 			)
 		)
-		(property "Footprint" ""
+		(property "Footprint" "Package_SO:SOIC-16_3.9x9.9mm_P1.27mm"
 			(at 96.52 162.56 0)
 			(effects

Commit message: tighten layout for final sizing
Parts:
- removed U103: 74LS04, Package_SO:SOIC-14_3.9x8.7mm_P1.27mm, symbol 74xx:74LS04
- added C38, C39, C40, C41, C42, C43, C44, C45, C46, C47, C48, C49, C50: 10nF, Capacitor_SMD:C_0603_1608Metric, symbol Device:C_Small
- added J48: OpMode, Connector_PinSocket_2.54mm:PinSocket_1x04_P2.54mm_Vertical, symbol Connector_Generic:Conn_01x04
- added J49: Default Palette, Connector_PinSocket_2.54mm:PinSocket_1x04_P2.54mm_Vertical, symbol Connector_Generic:Conn_01x04
- added J50: Output Palette, Connector_PinSocket_2.54mm:PinSocket_1x04_P2.54mm_Vertical, symbol Connector_Generic:Conn_01x04
- added J51: Triggers, Connector_PinSocket_2.54mm:PinSocket_1x04_P2.54mm_Vertical, symbol Connector_Generic:Conn_01x04
- added J52: Power and Clock, Connector_PinSocket_2.54mm:PinSocket_1x04_P2.54mm_Vertical, symbol Connector_Generic:Conn_01x04
- added J53: BDBus, Connector_PinHeader_2.54mm:PinHeader_1x08_P2.54mm_Vertical, symbol Connector_Generic:Conn_01x08
- added U136: 74LS04, Package_SO:SOIC-14_3.9x8.7mm_P1.27mm, symbol 74xx:74LS04
Connections:
- net BPP2Palette2 is gone; now on net BPP2Palette1: U40.11 (I1b)
- net +5V: now also C38.1, C39.1, C40.1, C41.1, C42.1, C43.1, C44.1, C45.1, C46.1, C47.1, C48.1, C49.1, C50.1, J52.1 (Pin_1), U136.14 (VCC)
- net BD0: now also J53.1 (Pin_1)
- net BD1: now also U30.18 (D7), J53.2 (Pin_2); no longer U30.4 (D1)
- net BD2: now also U30.4 (D1), J53.3 (Pin_3); no longer U30.7 (D2)
- net BD3: now also U30.17 (D6), J53.4 (Pin_4); no longer U30.8 (D3)
- net BD4: now also U30.14 (D5), J53.5 (Pin_5); no longer U30.13 (D4)
- net BD5: now also U30.7 (D2), J53.6 (Pin_6); no longer U30.14 (D5)
- net BD6: now also U30.8 (D3), J53.7 (Pin_7); no longer U30.17 (D6)
- net BD7: now also U30.13 (D4), J53.8 (Pin_8); no longer U30.18 (D7)
- net BMPalette0: now also J50.1 (Pin_1)
- net BMPalette1: now also U40.9 (Zb), J50.2 (Pin_2); no longer U41.7 (Za)
- net BMPalette2: now also U41.7 (Za), J50.3 (Pin_3); no longer U40.9 (Zb)
- net BMPalette3: now also J50.4 (Pin_4)
- net BPP0: now also J48.1 (Pin_1)
- net BPP1: now also J48.2 (Pin_2)
- net BPP1Palette1: now also U40.10 (I0b), J49.2 (Pin_2); no longer U41.6 (I0a)
- net BPP2Palette1: no longer U35.6 (~{Z}), U41.5 (I1a)
- net BPP4Palette1: now also U40.12 (I2b); no longer U41.4 (I2a)
- net BPP4Palette2: now also U41.4 (I2a); no longer U40.12 (I2b)
- net D1: now also U30.19 (O7); no longer U30.5 (O1)
- net D2: now also U30.5 (O1); no longer U30.6 (O2)
- net D3: now also U30.16 (O6); no longer U30.9 (O3)
- net D4: now also U30.15 (O5); no longer U30.12 (O4)
- net D5: now also U30.6 (O2); no longer U30.15 (O5)
- net D6: now also U30.9 (O3); no longer U30.16 (O6)
- net D7: now also U30.12 (O4); no longer U30.19 (O7)
- net DefaultPalette0: now also J49.1 (Pin_1)
- net GND: now also C38.2, C39.2, C40.2, C41.2, C42.2, C43.2, C44.2, C45.2, C46.2, C47.2, C48.2, C49.2, C50.2, J52.2 (Pin_2), J52.3 (Pin_3), U136.7 (GND); no longer U40.10 (I0b), U41.10 (I0b)
- net LoadPixelData: now also J51.1 (Pin_1)
- net PixelClock: now also J51.2 (Pin_2)
- net ~{HCountEnable}: now also J51.3 (Pin_3), U136.1
- net ~{MR}: now also U136.2
- net BPP2Palette3 renamed BPP1Palette3
- net BPP1Palette3: now also U41.10 (I0b), J49.4 (Pin_4)
- new net BPP1Palette2: J49.3 (Pin_3), U41.5 (I1a), U41.6 (I0a)
- no-connect marks 44 -> 48
