File: BitmapDataCounter.kicad_sch (KiCad schematic)
At the start: 5 parts, among them U21 74LS163, U22 74LS253, U23 74LS163, U24 74LS253, U8 74LS14

Commit message: provide annotation on modules
Connections:
- net +5V: now also U22.15 (OEb), U24.15 (OEb); no longer U24.1 (OEa)
- net GND: now also U24.1 (OEa); no longer U22.15 (OEb), U24.15 (OEb)
- net LoadEnable: no longer U22.1 (OEa)
- net ~{HLoadEnable}: now also U22.1 (OEa)
Changed lines of the file:
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@@
+		)
+	)
+	(text_box "U21 counts raw clock ticks and acts as a clock divider to reduce the clock by 2, 4, 8 or 16\n\nHLoadEnable is a continuous signal, the duration of which is the width of the viewport"
+		(exclude_from_sim no)
+		(at 76.2 38.1 0)
+		(size 33.02 19.05)
+		(margins 0.9525 0.9525 0.9525 0.9525)
+		(stroke
+			(width -0.0001)
+			(type solid)
+		)
+		(fill
+			(type none)
+		)
+		(effects
+			(font
+				(size 1.27 1.27)
+			)
+			(justify left top)
+		)
+	)
+	(text_box "U23 is the effective counter in this circuit, counting pixels"
+		(exclude_from_sim no)
+		(at 170.18 38.1 0)
+		(size 30.48 10.16)
+		(margins 0.9525 0.9525 0.9525 0.9525)
+		(stroke
+			(width -0.0001)
+			(type solid)
+		)
+		(fill
+			(type none)
+		)
+		(effects
+			(font
+				(size 1.27 1.27)
+			)
+			(justify left top)
+		)
+	)
+	(text_box "The BitmapDataCounter module defines when the BitmapPixelData module needs to load a fresh byte of data from the bitmap data bus\n\nTo do calculate when to load the module needs to run a separate counter clocked off the same source as the main pixel counter\nThe ViewPort module contains a trigger to start the counter out of phase with the data boundary so the data is correctly loaded in advance. Note this does not trigger the memory access, that requires another trigger event in another phase so that the data bus can be prepared before the load action takes place\n\nThe number of clock ticks per pixel and bits per pixel both impact how frequently the load signal fires. In this simplified design the faster timing options are not used but can be implemented from this design if needed"
+		(exclude_from_sim no)
+		(at 31.75 151.13 0)
+		(size 66.04 36.83)
+		(margins 0.9525 0.9525 0.9525 0.9525)
+		(stroke
+			(width 0)
+			(type solid)
+		)
+		(fill
+			(type color)
+			(color 255 255 255 1)
+		)
+		(effects
+			(font
+				(size 1.27 1.27)
+			)
+			(justify left top)
+		)
+	)
+	(text_box "The final stage, U24 selects which pixel count is the effective load pixel data trigger based on the bits per pixel. Note the clock order is reversed as 1 bit per pixel needs more clocks before loading data than 4 bits per pixel"
+		(exclude_from_sim no)
+		(at 217.17 38.1 0)
+		(size 33.02 20.32)
+		(margins 0.9525 0.9525 0.9525 0.9525)
+		(stroke
+			(width -0.0001)
+			(type solid)
+		)
+		(fill
+			(type none)
+		)
+		(effects
+			(font
+				(size 1.27 1.27)
+			)
+			(justify left top)
+		)
+	)
+	(text_box "U22 selects the effective clock division based on the clocks per pixel input"
+		(exclude_from_sim no)
+		(at 124.46 38.1 0)
+		(size 29.21 10.16)
+		(margins 0.9525 0.9525 0.9525 0.9525)
+		(stroke
+			(width -0.0001)
+			(type solid)
+		)
+		(fill
+			(type none)
+		)
+		(effects
+			(font
+				(size 1.27 1.27)
+			)
+			(justify left top)
 		)
 	)
@@
 	)
 	(junction
-		(at 220.98 97.79)
-		(diameter 0)
-		(color 0 0 0 0)
-	)
-	(junction
 		(at 71.12 91.44)
 		(diameter 0)
@@
 	)
 	(junction
+		(at 220.98 85.09)
+		(diameter 0)
+		(color 0 0 0 0)
+	)
+	(junction
 		(at 172.72 87.63)
 		(diameter 0)
@@
 	)
 	(junction
-		(at 127 99.06)
-		(diameter 0)
-		(color 0 0 0 0)
-	)
-	(junction
 		(at 220.98 90.17)
 		(diameter 0)
@@
 	(wire
 		(pts
+			(xy 123.19 104.14) (xy 127 104.14)
+		)
+		(stroke
+			(width 0)
+			(type default)
+		)
+	)
+	(wire
+		(pts
+			(xy 220.98 85.09) (xy 220.98 90.17)
+		)
+		(stroke
+			(width 0)
+			(type default)
+		)
+	)
+	(wire
+		(pts
+			(xy 217.17 102.87) (xy 220.98 102.87)
+		)
+		(stroke
+			(width 0)
+			(type default)
+		)
+	)
+	(wire
+		(pts
 			(xy 38.1 85.09) (xy 40.64 85.09)
 		)
@@
 	(wire
 		(pts
-			(xy 217.17 90.17) (xy 220.98 90.17)
+			(xy 217.17 85.09) (xy 220.98 85.09)
 		)
 		(stroke
@@
 	(wire
 		(pts
-			(xy 73.66 88.9) (xy 80.01 88.9)
+			(xy 76.2 88.9) (xy 80.01 88.9)
 		)
 		(stroke
@@
 	(wire
 		(pts
-			(xy 127 99.06) (xy 127 104.14)
-		)
-		(stroke
-			(width 0)
-			(type default)
-		)
-	)
-	(wire
-		(pts
 			(xy 123.19 91.44) (xy 127 91.44)
 		)
@@
 	(wire
 		(pts
-			(xy 220.98 97.79) (xy 220.98 102.87)
-		)
-		(stroke
-			(width 0)
-			(type default)
-		)
-	)
-	(wire
-		(pts
 			(xy 168.91 87.63) (xy 172.72 87.63)
 		)
@@
 		(pts
 			(xy 35.56 63.5) (xy 35.56 66.04)
-		)
-		(stroke
-			(width 0)
-			(type default)
-		)
-	)
-	(wire
-		(pts
-			(xy 213.36 85.09) (xy 220.98 85.09)
 		)
 		(stroke
@@
 			)
 			(justify left bottom)
-		)
-	)
-	(label "LoadEnable"
-		(at 127 86.36 180)
-		(effects
-			(font
-				(size 1.27 1.27)
-			)
-			(justify right bottom)
 		)
 	)
@@
 		)
 	)
+	(global_label "~{HLoadEnable}"
+		(shape input)
+		(at 127 86.36 180)
+		(fields_autoplaced yes)
+		(effects
+			(font
+				(size 1.27 1.27)
+			)
+			(justify right)
+		)
+		(property "Intersheetrefs" "${INTERSHEET_REFS}"
+			(at 111.8594 86.36 0)
+			(effects
+				(font
+					(size 1.27 1.27)
+				)
+				(justify right)
+				(hide yes)
+			)
+		)
+	)
 	(global_label "LoadPixelData"
 		(shape output)
@@
 	(symbol
 		(lib_id "power:+5V")
-		(at 213.36 85.09 0)
+		(at 217.17 102.87 0)
 		(unit 1)
 		(exclude_from_sim no)
@@
 		(dnp no)
 		(fields_autoplaced yes)
-		(property "Reference" "#PWR071"
-			(at 213.36 88.9 0)
+		(property "Reference" "#PWR0360"
+			(at 217.17 106.68 0)
 			(effects
 				(font
@@
 		)
 		(property "Value" "+5V"
-			(at 213.36 80.01 0)
+			(at 217.17 97.79 0)
 			(effects
 				(font
@@
 		)
 		(property "Footprint" ""
-			(at 213.36 85.09 0)
+			(at 217.17 102.87 0)
 			(effects
 				(font
@@
 		)
 		(property "Datasheet" ""
-			(at 213.36 85.09 0)
+			(at 217.17 102.87 0)
 			(effects
 				(font
@@
 		)
 		(property "Description" "Power symbol creates a global label with name \"+5V\""
-			(at 213.36 85.09 0)
+			(at 217.17 102.87 0)
 			(effects
 				(font
@@
 			(project "DIY-Video"
 				(path "/6c4ef05c-ecf5-4bee-ae4e-d72f13738678/ea58d469-cf1f-4bb0-82ac-67bd50353b02"
-					(reference "#PWR071")
+					(reference "#PWR0360")
 					(unit 1)
 				)
@@
 	(symbol
 		(lib_id "power:GND")
-		(at 217.17 90.17 0)
+		(at 217.17 85.09 0)
 		(unit 1)
 		(exclude_from_sim no)
@@
 		(fields_autoplaced yes)
 		(property "Reference" "#PWR068"
-			(at 217.17 96.52 0)
+			(at 217.17 91.44 0)
 			(effects
 				(font
@@
 		)
 		(property "Value" "GND"
-			(at 217.17 95.25 0)
+			(at 217.17 90.17 0)
 			(effects
 				(font
@@
 		)
 		(property "Footprint" ""
-			(at 217.17 90.17 0)
+			(at 217.17 85.09 0)
 			(effects
 				(font
@@
 		)
 		(property "Datasheet" ""
-			(at 217.17 90.17 0)
+			(at 217.17 85.09 0)
 			(effects
 				(font
@@
 		)
 		(property "Description" "Power symbol creates a global label with name \"GND\" , ground"
-			(at 217.17 90.17 0)
+			(at 217.17 85.09 0)
 			(effects
 				(font
@@
 	(symbol
 		(lib_id "power:+5V")
-		(at 73.66 88.9 0)
+		(at 76.2 88.9 0)
 		(unit 1)
 		(exclude_from_sim no)
@@
 		(fields_autoplaced yes)
 		(property "Reference" "#PWR059"
-			(at 73.66 92.71 0)
+			(at 76.2 92.71 0)
 			(effects
 				(font
@@
 		)
 		(property "Value" "+5V"
-			(at 73.66 83.82 0)
+			(at 76.2 83.82 0)
 			(effects
 				(font
@@
 		)
 		(property "Footprint" ""
-			(at 73.66 88.9 0)
+			(at 76.2 88.9 0)
 			(effects
 				(font
@@
 		)
 		(property "Datasheet" ""
-			(at 73.66 88.9 0)
+			(at 76.2 88.9 0)
 			(effects
 				(font
@@
 		)
 		(property "Description" "Power symbol creates a global label with name \"+5V\""
-			(at 73.66 88.9 0)
+			(at 76.2 88.9 0)
 			(effects
 				(font
@@
 					(unit 1)
 				)
+			)
+		)
+	)
+	(symbol
+		(lib_id "power:+5V")
+		(at 123.19 104.14 0)
+		(unit 1)
+		(exclude_from_sim no)
+		(in_bom yes)
+		(on_board yes)
+		(dnp no)
+		(fields_autoplaced yes)
+		(property "Reference" "#PWR0359"
+			(at 123.19 107.95 0)
+			(effects
+				(font
+					(size 1.27 1.27)
+				)
+				(hide yes)
+			)
+		)
+		(property "Value" "+5V"
+			(at 123.19 99.06 0)
+			(effects
+				(font
+					(size 1.27 1.27)
+				)
+			)
+		)
+		(property "Footprint" ""
+			(at 123.19 104.14 0)
+			(effects
+				(font
+					(size 1.27 1.27)
+				)
+				(hide yes)
+			)
+		)
+		(property "Datasheet" ""
+			(at 123.19 104.14 0)
+			(effects
+				(font
+					(size 1.27 1.27)
+				)
+				(hide yes)
+			)
+		)
+		(property "Description" "Power symbol creates a global label with name \"+5V\""
+			(at 123.19 104.14 0)
+			(effects
+				(font
+					(size 1.27 1.27)
+				)
+				(hide yes)
+			)
+		)
+		(pin "1"
+		)
+		(instances
+			(project "DIY-Video"
+				(path "/6c4ef05c-ecf5-4bee-ae4e-d72f13738678/ea58d469-cf1f-4bb0-82ac-67bd50353b02"
+					(reference "#PWR0359")
+					(unit 1)
+				)

Commit message: isolate each schematic function for testing
Parts:
- removed U8: 74LS14, Package_SO:SO-14_3.9x8.65mm_P1.27mm, symbol 74xx:74LS14
- added U118: 74LS04, Package_SO:SOIC-14_3.9x8.7mm_P1.27mm, symbol 74xx:74LS04
Connections:
- net LoadEnable: now also U118.2
- net ~{HLoadEnable}: now also U118.1

Commit message: rework schematic isolation
Parts:
- added J16: Power and Clock, Connector_PinSocket_2.54mm:PinSocket_1x04_P2.54mm_Vertical, symbol Connector_Generic:Conn_01x04
- added J17: Triggers, Connector_PinSocket_2.54mm:PinSocket_1x04_P2.54mm_Vertical, symbol Connector_Generic:Conn_01x04
- added J18: OpMode, Connector_PinSocket_2.54mm:PinSocket_1x04_P2.54mm_Vertical, symbol Connector_Generic:Conn_01x04
Connections:
- net +5V: now also U118.14 (VCC), J16.1 (Pin_1)
- net 14M: now also J16.4 (Pin_4)
- net BPP0: now also J18.1 (Pin_1)
- net BPP1: now also J18.2 (Pin_2)
- net CPP0: now also J18.3 (Pin_3)
- net CPP1: now also J18.4 (Pin_4)
- net GND: now also U118.7 (GND), J16.2 (Pin_2), J16.3 (Pin_3), J17.1 (Pin_1), J17.3 (Pin_3)
- net LoadPixelData: now also J17.4 (Pin_4)
- net ~{HLoadEnable}: now also J17.2 (Pin_2)

Commit message: tighten layout for final sizing
Parts:
- added C28, C29, C30, C31, C32: 10nF, Capacitor_SMD:C_0603_1608Metric, symbol Device:C_Small
Connections:
- net +5V: now also C28.1, C29.1, C30.1, C31.1, C32.1
- net GND: now also C28.2, C29.2, C30.2, C31.2, C32.2
