File: BitmapPixelCounter.kicad_sch (KiCad schematic)
At the start: 5 parts, among them U25 74LS14, U26 74LS163, U27 74LS253, U28 74LS163, U29 74LS253

Commit message: provide annotation on modules
Connections:
- net +5V: now also U27.15 (OEb), U29.15 (OEb); no longer U29.1 (OEa)
- net CountEnable: no longer U27.1 (OEa)
- net GND: now also U29.1 (OEa); no longer U27.15 (OEb), U29.15 (OEb)
- net ~{HCountEnable}: now also U27.1 (OEa)
Changed lines of the file:
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@@
+		)
+	)
+	(text_box "The BitmapPixelCounter module is effectively a copy of BitmapDataCounter but uses a different enable signal, starting at the first visible pixel of the viewport rather than before that point\n\nPotentially the two modules could be combined using an inverse of the \"load\" signal to trigger the pixel count but is likely to create a more complex solution than just repeating the four ICs here"
+		(exclude_from_sim no)
+		(at 21.59 153.67 0)
+		(size 66.04 36.83)
+		(margins 0.9525 0.9525 0.9525 0.9525)
+		(stroke
+			(width 0)
+			(type solid)
+		)
+		(fill
+			(type color)
+			(color 255 255 255 1)
+		)
+		(effects
+			(font
+				(size 1.27 1.27)
+			)
+			(justify left top)
 		)
 	)
@@
 	)
 	(junction
-		(at 218.44 107.95)
-		(diameter 0)
-		(color 0 0 0 0)
-	)
-	(junction
 		(at 218.44 102.87)
 		(diameter 0)
@@
 	)
 	(junction
+		(at 218.44 95.25)
+		(diameter 0)
+		(color 0 0 0 0)
+	)
+	(junction
 		(at 124.46 101.6)
 		(diameter 0)
@@
 	)
 	(junction
-		(at 124.46 109.22)
-		(diameter 0)
-		(color 0 0 0 0)
-	)
-	(junction
 		(at 218.44 100.33)
 		(diameter 0)
@@
 	(wire
 		(pts
-			(xy 214.63 100.33) (xy 218.44 100.33)
-		)
-		(stroke
-			(width 0)
-			(type default)
-		)
-	)
-	(wire
-		(pts
-			(xy 210.82 95.25) (xy 218.44 95.25)
+			(xy 214.63 95.25) (xy 218.44 95.25)
 		)
 		(stroke
@@
 		)
 	)
+	(wire
+		(pts
+			(xy 214.63 113.03) (xy 218.44 113.03)
+		)
+		(stroke
+			(width 0)
+			(type default)
+		)
+	)
 	(bus
 		(pts
@@
 	(wire
 		(pts
-			(xy 124.46 109.22) (xy 124.46 114.3)
-		)
-		(stroke
-			(width 0)
-			(type default)
-		)
-	)
-	(wire
-		(pts
 			(xy 124.46 101.6) (xy 124.46 104.14)
 		)
@@
 	(wire
 		(pts
-			(xy 218.44 107.95) (xy 218.44 113.03)
-		)
-		(stroke
-			(width 0)
-			(type default)
-		)
-	)
-	(wire
-		(pts
 			(xy 166.37 82.55) (xy 170.18 82.55)
 		)
@@
 	(wire
 		(pts
+			(xy 218.44 95.25) (xy 218.44 100.33)
+		)
+		(stroke
+			(width 0)
+			(type default)
+		)
+	)
+	(wire
+		(pts
 			(xy 68.58 101.6) (xy 77.47 101.6)
 		)
@@
 		(pts
 			(xy 35.56 81.28) (xy 38.1 81.28)
+		)
+		(stroke
+			(width 0)
+			(type default)
+		)
+	)
+	(wire
+		(pts
+			(xy 120.65 114.3) (xy 124.46 114.3)
 		)
 		(stroke
@@
 			)
 			(justify left bottom)
-		)
-	)
-	(label "CountEnable"
-		(at 124.46 96.52 180)
-		(effects
-			(font
-				(size 1.27 1.27)
-			)
-			(justify right bottom)
 		)
 	)
@@
 				)
 				(justify left)
+				(hide yes)
+			)
+		)
+	)
+	(global_label "~{HCountEnable}"
+		(shape input)
+		(at 124.46 96.52 180)
+		(fields_autoplaced yes)
+		(effects
+			(font
+				(size 1.27 1.27)
+			)
+			(justify right)
+		)
+		(property "Intersheetrefs" "${INTERSHEET_REFS}"
+			(at 108.3518 96.52 0)
+			(effects
+				(font
+					(size 1.27 1.27)
+				)
+				(justify right)
 				(hide yes)
 			)
@@
 	)
 	(symbol
+		(lib_id "power:+5V")
+		(at 214.63 113.03 0)
+		(unit 1)
+		(exclude_from_sim no)
+		(in_bom yes)
+		(on_board yes)
+		(dnp no)
+		(fields_autoplaced yes)
+		(property "Reference" "#PWR071"
+			(at 214.63 116.84 0)
+			(effects
+				(font
+					(size 1.27 1.27)
+				)
+				(hide yes)
+			)
+		)
+		(property "Value" "+5V"
+			(at 214.63 107.95 0)
+			(effects
+				(font
+					(size 1.27 1.27)
+				)
+			)
+		)
+		(property "Footprint" ""
+			(at 214.63 113.03 0)
+			(effects
+				(font
+					(size 1.27 1.27)
+				)
+				(hide yes)
+			)
+		)
+		(property "Datasheet" ""
+			(at 214.63 113.03 0)
+			(effects
+				(font
+					(size 1.27 1.27)
+				)
+				(hide yes)
+			)
+		)
+		(property "Description" "Power symbol creates a global label with name \"+5V\""
+			(at 214.63 113.03 0)
+			(effects
+				(font
+					(size 1.27 1.27)
+				)
+				(hide yes)
+			)
+		)
+		(pin "1"
+		)
+		(instances
+			(project "DIY-Video"
+				(path "/6c4ef05c-ecf5-4bee-ae4e-d72f13738678/935d5772-4398-4369-8a3a-93d8947ae994"
+					(reference "#PWR071")
+					(unit 1)
+				)
+			)
+		)
+	)
+	(symbol
 		(lib_id "power:GND")
-		(at 214.63 100.33 0)
+		(at 214.63 95.25 0)
 		(unit 1)
 		(exclude_from_sim no)
@@
 		(fields_autoplaced yes)
 		(property "Reference" "#PWR084"
-			(at 214.63 106.68 0)
+			(at 214.63 101.6 0)
 			(effects
 				(font
@@
 		)
 		(property "Value" "GND"
-			(at 214.63 105.41 0)
+			(at 214.63 100.33 0)
 			(effects
 				(font
@@
 		)
 		(property "Footprint" ""
-			(at 214.63 100.33 0)
+			(at 214.63 95.25 0)
 			(effects
 				(font
@@
 		)
 		(property "Datasheet" ""
-			(at 214.63 100.33 0)
+			(at 214.63 95.25 0)
 			(effects
 				(font
@@
 		)
 		(property "Description" "Power symbol creates a global label with name \"GND\" , ground"
-			(at 214.63 100.33 0)
+			(at 214.63 95.25 0)
 			(effects
 				(font
@@
 				(path "/6c4ef05c-ecf5-4bee-ae4e-d72f13738678/935d5772-4398-4369-8a3a-93d8947ae994"
 					(reference "#PWR084")
-					(unit 1)
-				)
-			)
-		)
-	)
-	(symbol
-		(lib_id "power:+5V")
-		(at 210.82 95.25 0)
-		(unit 1)
-		(exclude_from_sim no)
-		(in_bom yes)
-		(on_board yes)
-		(dnp no)
-		(fields_autoplaced yes)
-		(property "Reference" "#PWR083"
-			(at 210.82 99.06 0)
-			(effects
-				(font
-					(size 1.27 1.27)
-				)
-				(hide yes)
-			)
-		)
-		(property "Value" "+5V"
-			(at 210.82 90.17 0)
-			(effects
-				(font
-					(size 1.27 1.27)
-				)
-			)
-		)
-		(property "Footprint" ""
-			(at 210.82 95.25 0)
-			(effects
-				(font
-					(size 1.27 1.27)
-				)
-				(hide yes)
-			)
-		)
-		(property "Datasheet" ""
-			(at 210.82 95.25 0)
-			(effects
-				(font
-					(size 1.27 1.27)
-				)
-				(hide yes)
-			)
-		)
-		(property "Description" "Power symbol creates a global label with name \"+5V\""
-			(at 210.82 95.25 0)
-			(effects
-				(font
-					(size 1.27 1.27)
-				)
-				(hide yes)
-			)
-		)
-		(pin "1"
-		)
-		(instances
-			(project "DIY-Video"
-				(path "/6c4ef05c-ecf5-4bee-ae4e-d72f13738678/935d5772-4398-4369-8a3a-93d8947ae994"
-					(reference "#PWR083")
 					(unit 1)
 				)
@@
 					(unit 1)
 				)
+			)
+		)
+	)
+	(symbol
+		(lib_id "power:+5V")
+		(at 120.65 114.3 0)
+		(unit 1)
+		(exclude_from_sim no)
+		(in_bom yes)
+		(on_board yes)
+		(dnp no)
+		(fields_autoplaced yes)
+		(property "Reference" "#PWR083"
+			(at 120.65 118.11 0)
+			(effects
+				(font
+					(size 1.27 1.27)
+				)
+				(hide yes)
+			)
+		)
+		(property "Value" "+5V"
+			(at 120.65 109.22 0)
+			(effects
+				(font
+					(size 1.27 1.27)
+				)
+			)
+		)
+		(property "Footprint" ""
+			(at 120.65 114.3 0)
+			(effects
+				(font
+					(size 1.27 1.27)
+				)
+				(hide yes)
+			)
+		)
+		(property "Datasheet" ""
+			(at 120.65 114.3 0)
+			(effects
+				(font
+					(size 1.27 1.27)
+				)
+				(hide yes)
+			)
+		)
+		(property "Description" "Power symbol creates a global label with name \"+5V\""
+			(at 120.65 114.3 0)
+			(effects
+				(font
+					(size 1.27 1.27)
+				)
+				(hide yes)
+			)
+		)
+		(pin "1"
+		)
+		(instances
+			(project "DIY-Video"
+				(path "/6c4ef05c-ecf5-4bee-ae4e-d72f13738678/935d5772-4398-4369-8a3a-93d8947ae994"
+					(reference "#PWR083")
+					(unit 1)
+				)

Commit message: rework schematic isolation
Parts:
- removed U25: 74LS14, Package_SO:SO-14_3.9x8.65mm_P1.27mm, symbol 74xx:74LS14
- added U128: 74LS04, Package_SO:SOIC-14_3.9x8.7mm_P1.27mm, symbol 74xx:74LS04
Connections:
- net +5V: now also U128.14 (VCC)
- net CountEnable: now also U128.2
- net GND: now also U128.7 (GND)
- net ~{HCountEnable}: now also U128.1

Commit message: refine main board layout
Parts:
- added J45: Power and Clock, Connector_PinSocket_2.54mm:PinSocket_1x04_P2.54mm_Vertical, symbol Connector_Generic:Conn_01x04
- added J46: Triggers, Connector_PinSocket_2.54mm:PinSocket_1x04_P2.54mm_Vertical, symbol Connector_Generic:Conn_01x04
- added J47: OpMode, Connector_PinSocket_2.54mm:PinSocket_1x04_P2.54mm_Vertical, symbol Connector_Generic:Conn_01x04
Connections:
- net +5V: now also J45.1 (Pin_1)
- net 14M: now also J45.4 (Pin_4)
- net BPP0: now also J47.1 (Pin_1)
- net BPP1: now also J47.2 (Pin_2)
- net CPP0: now also J47.3 (Pin_3)
- net CPP1: now also J47.4 (Pin_4)
- net GND: now also J45.2 (Pin_2), J45.3 (Pin_3), J46.1 (Pin_1), J46.3 (Pin_3)
- net PixelClock: now also J46.4 (Pin_4)
- net ~{HCountEnable}: now also J46.2 (Pin_2)

Commit message: tighten layout for final sizing
Parts:
- added C33, C34, C35, C36, C37: 10nF, Capacitor_SMD:C_0603_1608Metric, symbol Device:C_Small
Connections:
- net +5V: now also C33.1, C34.1, C35.1, C36.1, C37.1
- net GND: now also C33.2, C34.2, C35.2, C36.2, C37.2
- net PT0: now also U29.3 (I3a); no longer U29.6 (I0a)
- net PT1: now also U29.4 (I2a); no longer U29.5 (I1a)
- net PT2: now also U29.5 (I1a); no longer U29.4 (I2a)
- net PT3: now also U29.6 (I0a); no longer U29.3 (I3a)
