File: controlRegisters.kicad_sch (KiCad schematic)
At the start: 19 parts, among them U67 74LS32, U76 74LS04, U83 74LS08, U84 74LS374, U85 74LS244, U86 74LS374, U87 74LS244, U88 74LS374, U89 74LS244, U90 74LS08, U91 74LS21, U92 74LS21, U93 74LS32, U94 74LS32, U95 74LS32, U96 74LS374, U97 74LS244, U98 74LS32, U99 74LS32

Commit message: refine bus contention solution for host interface
Changed lines of the file:
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@@
+		)
+	)
+	(text_box "~{ExtAdd} flags when the host is making *any* read or write request\n\nThis is gated against the different device select channels\n~{IntMem} is specifically the bitmap memory"
+		(exclude_from_sim no)
+		(at 35.56 102.87 0)
+		(size 41.91 17.78)
+		(margins 0.9525 0.9525 0.9525 0.9525)
+		(stroke
+			(width 0)
+			(type solid)
+		)
+		(fill
+			(type none)
+		)
+		(effects
+			(font
+				(size 1.27 1.27)
+			)
+			(justify left top)
 		)
 	)

Commit message: rework schematic isolation
Parts:
- removed U67, U95, U99: 74LS32, Package_SO:SO-14_3.9x8.65mm_P1.27mm, symbol 74xx:74LS32
- removed U91, U92: 74LS21, Package_SO:SO-14_3.9x8.65mm_P1.27mm, symbol 74xx:74LS21
- added J19, J20, J22, J23, J25, J26, J28, J29: XDBus, Connector_PinHeader_1.27mm:PinHeader_1x08_P1.27mm_Vertical, symbol Connector_Generic:Conn_01x08
- added J21: Register0, Connector_PinHeader_1.27mm:PinHeader_1x10_P1.27mm_Vertical, symbol Connector_Generic:Conn_01x10
- added J24: Register2, Connector_PinHeader_1.27mm:PinHeader_1x10_P1.27mm_Vertical, symbol Connector_Generic:Conn_01x10
- added J27: Register1, Connector_PinHeader_1.27mm:PinHeader_1x10_P1.27mm_Vertical, symbol Connector_Generic:Conn_01x10
- added J30: Register3, Connector_PinHeader_1.27mm:PinHeader_1x10_P1.27mm_Vertical, symbol Connector_Generic:Conn_01x10
- added U25: 74LS32, Package_SO:SOIC-14_3.9x8.7mm_P1.27mm, symbol 74xx:74LS32
- added U67: 74LS138, Package_SO:SOIC-16_3.9x9.9mm_P1.27mm, symbol 74xx:74LS138
Connections:
- net +5V: now also U25.14 (VCC), U67.16 (VCC)
- net A0: now also U67.1 (A0)
- net A1: now also U67.2 (A1)
- net A2: now also U67.3 (A2)
- net BPP0: now also J21.5 (Pin_5)
- net BPP1: now also J21.6 (Pin_6)
- net Border0: now also J24.1 (Pin_1)
- net Border1: now also J24.2 (Pin_2)
- net Border2: now also J24.3 (Pin_3)
- net Border3: now also J24.4 (Pin_4)
- net CPP0: now also J21.7 (Pin_7)
- net CPP1: now also J21.8 (Pin_8)
- net DevSel4: now also U67.6 (E3); no longer U93.1, U93.12, U94.12, U94.4
- net EnExternalTrigger: now also J24.8 (Pin_8)
- net EnableSprite: now also J30.2 (Pin_2)
- net EnableTile: now also J30.1 (Pin_1)
- net ExtTriggerHi/~{Lo}: now also J24.7 (Pin_7)
- net External: now also J24.6 (Pin_6)
- net FontMap0: now also J30.3 (Pin_3)
- net FontMap1: now also J30.4 (Pin_4)
- net Format: now also J24.5 (Pin_5)
- net GND: now also U25.7 (GND), U67.4 (E1), U67.5 (E2), U67.8 (GND)
- net Page13: now also U25.3
- net Page14: now also U25.6
- net PageSize0: now also J21.1 (Pin_1)
- net PageSize1: now also J21.2 (Pin_2)
- net PagedA13: now also J21.3 (Pin_3)
- net PagedA14: now also J21.4 (Pin_4)
- net RR0: now also J27.2 (Pin_2)
- net RR1: now also J27.3 (Pin_3)
- net VP~{Int}: now also J27.5 (Pin_5)
- net XD0: now also J19.1 (Pin_1), J20.1 (Pin_1), J22.1 (Pin_1), J23.1 (Pin_1), J25.1 (Pin_1), J26.1 (Pin_1), J28.1 (Pin_1), J29.1 (Pin_1)
- net XD1: now also J19.2 (Pin_2), J20.2 (Pin_2), J22.2 (Pin_2), J23.2 (Pin_2), J25.2 (Pin_2), J26.2 (Pin_2), J28.2 (Pin_2), J29.2 (Pin_2)
- net XD2: now also J19.3 (Pin_3), J20.3 (Pin_3), J22.3 (Pin_3), J23.3 (Pin_3), J25.3 (Pin_3), J26.3 (Pin_3), J28.3 (Pin_3), J29.3 (Pin_3)
- net XD3: now also J19.4 (Pin_4), J20.4 (Pin_4), J22.4 (Pin_4), J23.4 (Pin_4), J25.4 (Pin_4), J26.4 (Pin_4), J28.4 (Pin_4), J29.4 (Pin_4)
- net XD4: now also J19.5 (Pin_5), J20.5 (Pin_5), J22.5 (Pin_5), J23.5 (Pin_5), J25.5 (Pin_5), J26.5 (Pin_5), J28.5 (Pin_5), J29.5 (Pin_5)
- net XD5: now also J19.6 (Pin_6), J20.6 (Pin_6), J22.6 (Pin_6), J23.6 (Pin_6), J25.6 (Pin_6), J26.6 (Pin_6), J28.6 (Pin_6), J29.6 (Pin_6)
- net XD6: now also J19.7 (Pin_7), J20.7 (Pin_7), J22.7 (Pin_7), J23.7 (Pin_7), J25.7 (Pin_7), J26.7 (Pin_7), J28.7 (Pin_7), J29.7 (Pin_7)
- net XD7: now also J19.8 (Pin_8), J20.8 (Pin_8), J22.8 (Pin_8), J23.8 (Pin_8), J25.8 (Pin_8), J26.8 (Pin_8), J28.8 (Pin_8), J29.8 (Pin_8)
- net ~{A}/G: now also J27.1 (Pin_1)
- net ~{ExtRead}: now also U93.13, U94.13, U94.5; no longer U94.10
- net ~{ExtWrite}: now also U93.2, U94.10
- net ~{HSInt}: now also J27.6 (Pin_6)
- net ~{RPInt}: now also J27.8 (Pin_8)
- net ~{RegisterRead0}: now also J21.9 (Pin_9)
- net ~{RegisterRead1}: now also U93.11, J27.9 (Pin_9); no longer U94.8
- net ~{RegisterRead2}: now also U94.6, J24.9 (Pin_9)
- net ~{RegisterRead3}: now also U94.11, J30.9 (Pin_9)
- net ~{RegisterWrite0}: now also J21.10 (Pin_10)
- net ~{RegisterWrite1}: now also U93.3, J27.10 (Pin_10); no longer U94.3
- net ~{RegisterWrite2}: now also U94.8, J24.10 (Pin_10)
- net ~{RegisterWrite3}: now also U94.3, J30.10 (Pin_10)
- net ~{SelectRegister0}: now also U93.4, U93.9, U67.15 (O0); no longer U93.13, U94.5
- net ~{SelectRegister1}: now also U93.1, U93.12, U67.14 (O1); no longer U93.2, U94.13
- net ~{SelectRegister2}: now also U94.4, U94.9, U67.13 (O2)
- net ~{SelectRegister3}: now also U94.1, U94.12, U67.12 (O3)
- net ~{VPInt}: now also J27.4 (Pin_4)
- net ~{VSInt}: now also J27.7 (Pin_7)
- net at U90.6: now also U25.2
- net at U83.3: now also U25.1
- net R3B4: now reaches U96.12 (O4), U97.11 (I0b)
- net R3B4: now also J30.5 (Pin_5)
- net R3B5: now reaches U96.15 (O5), U97.13 (I1b)
- net R3B5: now also J30.6 (Pin_6)
- net R3B6: now reaches U96.16 (O6), U97.15 (I2b)
- net R3B6: now also J30.7 (Pin_7)
- net R3B7: now reaches U96.19 (O7), U97.17 (I3b)
- net R3B7: now also J30.8 (Pin_8)
- net at U90.11: now also U25.5
- net at U90.8: now also U25.4
- new net ~{SelectRegister4}: U67.11 (O4)
- new net ~{SelectRegister5}: U67.10 (O5)
- new net ~{SelectRegister6}: U67.9 (O6)
- new net ~{SelectRegister7}: U67.7 (O7)
Other:
- note added: "Register 3"
- moved on the sheet: U84, U85, U86, U87, U88, U89, U90E, U93B, U93C, U94E, U96, U97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

Commit message: spin register out as separate board
Parts:
- removed unit 1 of U76
- removed unit 4 of U83
- removed unit 2 of U83
- removed unit 3 of U83
- removed unit 1 of U98
- removed unit 2 of U98
- added J31, J32, J34, J35, J37, J38, J40, J41: XDBus, Connector_PinHeader_1.27mm:PinHeader_1x08_P1.27mm_Vertical, symbol Connector_Generic:Conn_01x08
- added J33: Register4, Connector_PinHeader_1.27mm:PinHeader_1x10_P1.27mm_Vertical, symbol Connector_Generic:Conn_01x10
- added J36: Register6, Connector_PinHeader_1.27mm:PinHeader_1x10_P1.27mm_Vertical, symbol Connector_Generic:Conn_01x10
- added J39: Register5, Connector_PinHeader_1.27mm:PinHeader_1x10_P1.27mm_Vertical, symbol Connector_Generic:Conn_01x10
- added J42: Register7, Connector_PinHeader_1.27mm:PinHeader_1x10_P1.27mm_Vertical, symbol Connector_Generic:Conn_01x10
- added U130, U132, U134, U95: 74LS244, Package_SO:SO-20_5.3x12.6mm_P1.27mm, symbol 74xx:74LS244
- added U131, U133, U92, U99: 74LS374, Package_SO:SO-20_5.3x12.6mm_P1.27mm, symbol 74xx:74LS374
- added U135: 74LS32, Package_SO:SOIC-14_3.9x8.7mm_P1.27mm, symbol 74xx:74LS32
- U67: value 74LS138 -> 74ALS138
Connections:
- net ~{ExtRead} is gone; now on net ~{ClkExtRead}: U93.13, U93.5, U94.13, U94.5
- net ~{ExtWrite} is gone; now on net ~{ClkExtWrite}: U93.10, U93.2, U94.10, U94.2
- net +5V: now also U130.20 (VCC), U131.20 (VCC), U132.20 (VCC), U133.20 (VCC), U134.20 (VCC), U135.14 (VCC), U92.20 (VCC), U95.20 (VCC), U99.20 (VCC)
- net A0: no longer U76.3
- net A1: no longer U76.11
- net GND: now also U130.10 (GND), U130.19 (OEb), U131.1 (OE), U131.10 (GND), U132.10 (GND), U132.19 (OEb), U133.1 (OE), U133.10 (GND), U134.10 (GND), U134.19 (OEb), U135.7 (GND), U92.1 (OE), U92.10 (GND), U95.10 (GND), U95.19 (OEb), U99.1 (OE), U99.10 (GND); no longer U67.5 (E2), U98.10, U98.12, U98.13, U98.9
- net XD0: now also J31.1 (Pin_1), J32.1 (Pin_1), J34.1 (Pin_1), J35.1 (Pin_1), J37.1 (Pin_1), J38.1 (Pin_1), J40.1 (Pin_1), J41.1 (Pin_1), U130.18 (O0a), U131.3 (D0), U132.18 (O0a), U133.3 (D0), U134.18 (O0a), U92.3 (D0), U95.18 (O0a), U99.3 (D0)
- net XD1: now also J31.2 (Pin_2), J32.2 (Pin_2), J34.2 (Pin_2), J35.2 (Pin_2), J37.2 (Pin_2), J38.2 (Pin_2), J40.2 (Pin_2), J41.2 (Pin_2), U130.16 (O1a), U131.4 (D1), U132.16 (O1a), U133.4 (D1), U134.16 (O1a), U92.4 (D1), U95.16 (O1a), U99.4 (D1)
- net XD2: now also J31.3 (Pin_3), J32.3 (Pin_3), J34.3 (Pin_3), J35.3 (Pin_3), J37.3 (Pin_3), J38.3 (Pin_3), J40.3 (Pin_3), J41.3 (Pin_3), U130.14 (O2a), U131.7 (D2), U132.14 (O2a), U133.7 (D2), U134.14 (O2a), U92.7 (D2), U95.14 (O2a), U99.7 (D2)
- net XD3: now also J31.4 (Pin_4), J32.4 (Pin_4), J34.4 (Pin_4), J35.4 (Pin_4), J37.4 (Pin_4), J38.4 (Pin_4), J40.4 (Pin_4), J41.4 (Pin_4), U130.12 (O3a), U131.8 (D3), U132.12 (O3a), U133.8 (D3), U134.12 (O3a), U92.8 (D3), U95.12 (O3a), U99.8 (D3)
- net XD4: now also J31.5 (Pin_5), J32.5 (Pin_5), J34.5 (Pin_5), J35.5 (Pin_5), J37.5 (Pin_5), J38.5 (Pin_5), J40.5 (Pin_5), J41.5 (Pin_5), U130.9 (O0b), U131.13 (D4), U132.9 (O0b), U133.13 (D4), U134.9 (O0b), U92.13 (D4), U95.9 (O0b), U99.13 (D4)
- net XD5: now also J31.6 (Pin_6), J32.6 (Pin_6), J34.6 (Pin_6), J35.6 (Pin_6), J37.6 (Pin_6), J38.6 (Pin_6), J40.6 (Pin_6), J41.6 (Pin_6), U130.7 (O1b), U131.14 (D5), U132.7 (O1b), U133.14 (D5), U134.7 (O1b), U92.14 (D5), U95.7 (O1b), U99.14 (D5)
- net XD6: now also J31.7 (Pin_7), J32.7 (Pin_7), J34.7 (Pin_7), J35.7 (Pin_7), J37.7 (Pin_7), J38.7 (Pin_7), J40.7 (Pin_7), J41.7 (Pin_7), U130.5 (O2b), U131.17 (D6), U132.5 (O2b), U133.17 (D6), U134.5 (O2b), U92.17 (D6), U95.5 (O2b), U99.17 (D6)
- net XD7: now also J31.8 (Pin_8), J32.8 (Pin_8), J34.8 (Pin_8), J35.8 (Pin_8), J37.8 (Pin_8), J38.8 (Pin_8), J40.8 (Pin_8), J41.8 (Pin_8), U130.3 (O3b), U131.18 (D7), U132.3 (O3b), U133.18 (D7), U134.3 (O3b), U92.18 (D7), U95.3 (O3b), U99.18 (D7)
- net ~{SelectRegister4}: now also U98.12, U98.9
- net ~{SelectRegister5}: now also U25.12, U25.9
- net ~{SelectRegister6}: now also U135.1, U135.4
- net ~{SelectRegister7}: now also U135.12, U135.9
- net ~{RegisterRead4}: now reaches U98.11
- net ~{RegisterRead4}: now also J33.9 (Pin_9), U95.1 (OEa)
- net ~{RegisterRead5}: now reaches U25.11
- net ~{RegisterRead5}: now also J39.9 (Pin_9), U132.1 (OEa)
- net ~{ClkExtRead}: now reaches U25.13
- net ~{ClkExtRead}: now also U98.13, U135.13, U135.5
- net ~{RegisterWrite4}: now reaches U98.8
- net ~{RegisterWrite4}: now also J33.10 (Pin_10), U92.11 (Cp)
- net ~{ClkExtWrite}: now reaches U25.10
- net ~{ClkExtWrite}: now also U98.10, U135.10, U135.2
- net ~{RegisterWrite5}: now reaches U25.8
- net ~{RegisterWrite5}: now also J39.10 (Pin_10), U131.11 (Cp)
- net ~{A0}: no longer names the net of U76.4
- net ~{A1}: no longer names the net of U76.10
- new net R4B0: J33.1 (Pin_1), U92.2 (O0), U95.2 (I0a)
- new net R4B1: J33.2 (Pin_2), U92.5 (O1), U95.4 (I1a)
- new net R4B2: J33.3 (Pin_3), U92.6 (O2), U95.6 (I2a)
- new net R4B3: J33.4 (Pin_4), U92.9 (O3), U95.8 (I3a)
- new net R4B4: J33.5 (Pin_5), U92.12 (O4), U95.11 (I0b)
- new net R4B5: J33.6 (Pin_6), U92.15 (O5), U95.13 (I1b)
- new net R4B6: J33.7 (Pin_7), U92.16 (O6), U95.15 (I2b)
- new net R4B7: J33.8 (Pin_8), U92.19 (O7), U95.17 (I3b)
- new net R5B0: J39.1 (Pin_1), U131.2 (O0), U132.2 (I0a)
- new net R5B1: J39.2 (Pin_2), U131.5 (O1), U132.4 (I1a)
- new net R5B2: J39.3 (Pin_3), U131.6 (O2), U132.6 (I2a)
- new net R5B3: J39.4 (Pin_4), U131.9 (O3), U132.8 (I3a)
- new net R5B4: J39.5 (Pin_5), U131.12 (O4), U132.11 (I0b)
- new net R5B5: J39.6 (Pin_6), U131.15 (O5), U132.13 (I1b)
- new net R5B6: J39.7 (Pin_7), U131.16 (O6), U132.15 (I2b)
- new net R5B7: J39.8 (Pin_8), U131.19 (O7), U132.17 (I3b)
- new net R6B0: J36.1 (Pin_1), U130.2 (I0a), U99.2 (O0)
- new net R6B1: J36.2 (Pin_2), U130.4 (I1a), U99.5 (O1)
- new net R6B2: J36.3 (Pin_3), U130.6 (I2a), U99.6 (O2)
- new net R6B3: J36.4 (Pin_4), U130.8 (I3a), U99.9 (O3)
- new net R6B4: J36.5 (Pin_5), U130.11 (I0b), U99.12 (O4)
- new net R6B5: J36.6 (Pin_6), U130.13 (I1b), U99.15 (O5)
- new net R6B6: J36.7 (Pin_7), U130.15 (I2b), U99.16 (O6)
- new net R6B7: J36.8 (Pin_8), U130.17 (I3b), U99.19 (O7)
- new net R7B0: J42.1 (Pin_1), U133.2 (O0), U134.2 (I0a)
- new net R7B1: J42.2 (Pin_2), U133.5 (O1), U134.4 (I1a)
- new net R7B2: J42.3 (Pin_3), U133.6 (O2), U134.6 (I2a)
- new net R7B3: J42.4 (Pin_4), U133.9 (O3), U134.8 (I3a)
- new net R7B4: J42.5 (Pin_5), U133.12 (O4), U134.11 (I0b)
- new net R7B5: J42.6 (Pin_6), U133.15 (O5), U134.13 (I1b)
- new net R7B6: J42.7 (Pin_7), U133.16 (O6), U134.15 (I2b)
- new net R7B7: J42.8 (Pin_8), U133.19 (O7), U134.17 (I3b)
- new net ~{RegBank0}: U67.5 (E2)
- new net ~{RegisterRead6}: J36.9 (Pin_9), U130.1 (OEa), U135.6
- new net ~{RegisterRead7}: J42.9 (Pin_9), U134.1 (OEa), U135.11
- new net ~{RegisterWrite6}: J36.10 (Pin_10), U135.3, U99.11 (Cp)
- new net ~{RegisterWrite7}: J42.10 (Pin_10), U133.11 (Cp), U135.8
- no-connect marks 3 -> 1
Other:
- note added: "Register 4"
- note added: "Register 5"
- note added: "Register 6"
- note added: "Register 7"
- moved on the sheet: J19, J20, J21, J22, J23, J24, J25, J26, J27, J28, J29, J30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

Commit message: tighten layout for final sizing
Parts:
- removed unit 1 of U83
- added unit 1 of U90
Connections:
- net A13: now also U90.2
- net ~{PageSize0}: now also U90.1
- net at U25.1: now also U90.3
