File: viewport.kicad_sch (KiCad schematic)
At the start: 35 parts, among them J43 Power, J5 posX, J6 posY, J7 ViewportTriggers, U11 74LS00, U112 74LS30, U113 74LS30, U114 74LS00, U115 74LS32, U117 74LS08, U119 74LS08, U12 74LS30, U13 74LS20, U14 74LS04, U15 74LS30, U16 74LS20, U17 74LS30, U18 74LS00, U19 74LS32, U20 74LS30

Commit message: tighten layout for final sizing
Parts:
- removed U117: 74LS08, Package_SO:SO-14_3.9x8.65mm_P1.27mm, symbol 74xx:74LS08
- added unit 1 of U119
Changed lines of the file:
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@@
+	)
+	(symbol
+		(lib_id "74xx:74LS08")
+		(at 316.23 99.06 0)
+		(unit 1)
+		(exclude_from_sim no)
+		(in_bom yes)
+		(on_board yes)
+		(dnp no)
+		(fields_autoplaced yes)
+		(property "Reference" "U119"
+			(at 316.2217 90.17 0)
+			(effects
+				(font
+					(size 1.27 1.27)
+				)
+			)
+		)
+		(property "Value" "74LS08"
+			(at 316.2217 92.71 0)
+			(effects
+				(font
+					(size 1.27 1.27)
+				)
+			)
+		)
+		(property "Footprint" ""
+			(at 316.23 99.06 0)
+			(effects
+				(font
+					(size 1.27 1.27)
+				)
+				(hide yes)
+			)
+		)
+		(property "Datasheet" "http://www.ti.com/lit/gpn/sn74LS08"
+			(at 316.23 99.06 0)
+			(effects
+				(font
+					(size 1.27 1.27)
+				)
+				(hide yes)
+			)
+		)
+		(property "Description" "Quad And2"
+			(at 316.23 99.06 0)
+			(effects
+				(font
+					(size 1.27 1.27)
+				)
+				(hide yes)
+			)
+		)
+		(pin "3"
+		)
+		(pin "8"
+		)
+		(pin "5"
+		)
+		(pin "2"
+		)
+		(pin "4"
+		)
+		(pin "6"
+		)
+		(pin "1"
+		)
+		(pin "9"
+		)
+		(pin "10"
+		)
+		(pin "14"
+		)
+		(pin "12"
+		)
+		(pin "11"
+		)
+		(pin "13"
+		)
+		(pin "7"
+		)
+		(instances
+			(project "DIY-Video"
+				(path "/6c4ef05c-ecf5-4bee-ae4e-d72f13738678/4023660c-3ec4-409a-be3a-58018e7d8eb1"
+					(reference "U119")
+					(unit 1)
+				)
+			)
+		)
 	)
 	(symbol
@@
 					(unit 1)
 				)
-			)
-		)
-	)
-	(symbol
-		(lib_id "74xx:74LS08")
-		(at 341.63 127 0)
-		(unit 1)
-		(exclude_from_sim no)
-		(in_bom yes)
-		(on_board yes)
-		(dnp no)
-		(fields_autoplaced yes)
-		(property "Reference" "U117"
-			(at 341.6217 118.11 0)
-			(effects
-				(font
-					(size 1.27 1.27)
-				)
-			)
-		)
-		(property "Value" "74LS08"
-			(at 341.6217 120.65 0)
-			(effects
-				(font
-					(size 1.27 1.27)
-				)
-			)
-		)
-		(property "Footprint" "Package_SO:SO-14_3.9x8.65mm_P1.27mm"
-			(at 341.63 127 0)
-			(effects
-				(font
-					(size 1.27 1.27)
-				)
-				(hide yes)
-			)
-		)
-		(property "Datasheet" "http://www.ti.com/lit/gpn/sn74LS08"
-			(at 341.63 127 0)
-			(effects
-				(font
-					(size 1.27 1.27)
-				)
-				(hide yes)
-			)
-		)
-		(property "Description" "Quad And2"
-			(at 341.63 127 0)
-			(effects
-				(font
-					(size 1.27 1.27)
-				)
-				(hide yes)
-			)
-		)
-		(pin "2"
-		)
-		(pin "3"
-		)
-		(pin "1"
-		)
-		(pin "11"
-		)
-		(pin "10"
-		)
-		(pin "5"
-		)
-		(pin "6"
-		)
-		(pin "4"
-		)
-		(pin "9"
-		)
-		(pin "8"
-		)
-		(pin "12"
-		)
-		(pin "13"
-		)
-		(pin "14"
-		)
-		(pin "7"
-		)
-		(instances
-			(project "DIY-Video"
-				(path "/6c4ef05c-ecf5-4bee-ae4e-d72f13738678/4023660c-3ec4-409a-be3a-58018e7d8eb1"
-					(reference "U117")
-					(unit 1)
-				)
