File: DIY-Register-Block/DIY-Register-Block.kicad_pcb (KiCad board)
At the start: 2 copper layers, 133.4 x 62 mm, 44 parts, among them J1 Register0, J10 XDBus, J11 XDBus, J12 Register3, J13 XDBus, J14 XDBus, J15 Register4, J16 XDBus, J17 XDBus, J18 Register5, J19 XDBus, J2 XDBus, J20 XDBus, J21 Register6, J22 XDBus, J23 XDBus, J24 Register7, J25 Control, J26 XDBus, J27 Reg0, J28 Reg1, J29 Reg2, J3 XDBus, J30 Reg3, J31 Reg4, J32 Reg5, J33 Reg6, J34 Reg7, J4 XDBus, J5 XDBus, J6 Register1, J7 XDBus, J8 XDBus, J9 Register2, U1 74ALS138, U2 74LS32, U3 74LS32, U4 74LS32, U5 74LS32

Commit message: refine main board layout
Parts:
- U5: footprint Package_SO:SOIC-14_3.9x8.7mm_P1.27mm -> Package_SO:SO-14_3.9x8.65mm_P1.27mm
- moved J31 1.17 mm to (103.3, 84.4)
- moved J32 1.17 mm to (103.3, 87.0)
Routing:
- net ~{ClkExtRead}: track 214.3 -> 215.2 mm
- net /~{SelectRegister1}: track 62.2 -> 61.3 mm
- net /~{RegisterWrite1}: track 24.7 -> 25.3 mm
- net /~{RegisterWrite3}: track 24.7 -> 25.3 mm
- net /~{RegisterWrite7}: track 24.7 -> 25.3 mm
- net /~{RegisterWrite5}: track 24.7 -> 25.3 mm
- net GND: vias 12 -> 154
- net /~{SelectRegister3}: vias 3 -> 2
- added copper zone on B.Cu, net GND
- added copper zone on F.Cu, net GND
